File: extras/kicad/motor_board.kicad2.kicad_sch (KiCad schematic)
At the start: 21 parts, among them J1 CONN_08NO_SILK_FEMALE_PTH, J2 CONN_08NO_SILK_FEMALE_PTH, J3 CONN_08NO_SILK_FEMALE_PTH, J4 CONN_08NO_SILK_FEMALE_PTH, J5 CONN_08{dblquote}, J6 CONN_08{dblquote}, J8 CONN_08{dblquote}, SW1 SPDT-HIGH-AMP-SWITCHPTH, X1 1751280, X2 1751280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

Commit message: Add files via upload
Connections:
- net MOTOR_L2_EN: now also J6.8; no longer J8.2
- net MOTOR_L2_IN1: now also J6.6; no longer J8.4
- net MOTOR_L2_IN2: now also J6.7; no longer J8.3
- net MOTOR_L2_OUT1: now also J5.4; no longer J?.7
- net MOTOR_L2_OUT2: now also J5.5; no longer J?.6
- net MOTOR_R1_EN: now also J8.2; no longer J6.8
- net MOTOR_R1_IN1: now also J8.4; no longer J6.6
- net MOTOR_R1_IN2: now also J8.3; no longer J6.7
- net MOTOR_R1_OUT1: now also J?.7; no longer J5.4
- net MOTOR_R1_OUT2: now also J?.6; no longer J5.5
Changed lines of the file:
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@@
     (effects (font (size 1.2446 1.2446)) (justify left bottom))
   )
-  (label "MOTOR_L2_EN" (at 55.88 80.01 0)
+  (label "MOTOR_R1_EN" (at 55.88 80.01 0)
     (effects (font (size 1.2446 1.2446)) (justify left bottom))
   )
@@
     (effects (font (size 1.2446 1.2446)) (justify left bottom))
   )
-  (label "MOTOR_R1_IN2" (at 111.76 68.58 0)
+  (label "MOTOR_L2_IN2" (at 111.76 68.58 0)
     (effects (font (size 1.2446 1.2446)) (justify left bottom))
   )
@@
     (effects (font (size 1.2446 1.2446)) (justify left bottom))
   )
-  (label "MOTOR_L2_OUT1" (at 21.59 80.01 0)
+  (label "MOTOR_R1_OUT1" (at 21.59 80.01 0)
     (effects (font (size 1.2446 1.2446)) (justify left bottom))
   )
@@
     (effects (font (size 1.2446 1.2446)) (justify left bottom))
   )
-  (label "MOTOR_L2_OUT2" (at 21.59 77.47 0)
+  (label "MOTOR_R1_OUT2" (at 21.59 77.47 0)
     (effects (font (size 1.2446 1.2446)) (justify left bottom))
   )
-  (label "MOTOR_R1_IN1" (at 111.76 71.12 0)
+  (label "MOTOR_L2_IN1" (at 111.76 71.12 0)
     (effects (font (size 1.2446 1.2446)) (justify left bottom))
   )
@@
     (effects (font (size 1.2446 1.2446)) (justify left bottom))
   )
-  (label "MOTOR_R1_OUT1" (at 76.2 73.66 0)
+  (label "MOTOR_L2_OUT1" (at 76.2 73.66 0)
     (effects (font (size 1.2446 1.2446)) (justify left bottom))
   )
@@
     (effects (font (size 1.2446 1.2446)) (justify left bottom))
   )
-  (label "MOTOR_L2_IN2" (at 55.88 77.47 0)
+  (label "MOTOR_R1_IN2" (at 55.88 77.47 0)
     (effects (font (size 1.2446 1.2446)) (justify left bottom))
   )
@@
     (effects (font (size 1.2446 1.2446)) (justify left bottom))
   )
-  (label "MOTOR_R1_EN" (at 111.76 66.04 0)
+  (label "MOTOR_L2_EN" (at 111.76 66.04 0)
     (effects (font (size 1.2446 1.2446)) (justify left bottom))
   )
@@
     (effects (font (size 1.2446 1.2446)) (justify left bottom))
   )
-  (label "MOTOR_R1_OUT2" (at 77.47 76.2 0)
+  (label "MOTOR_L2_OUT2" (at 77.47 76.2 0)
     (effects (font (size 1.2446 1.2446)) (justify left bottom))
   )
@@
     (effects (font (size 1.2446 1.2446)) (justify left bottom))
   )
-  (label "MOTOR_L2_IN1" (at 55.88 74.93 0)
+  (label "MOTOR_R1_IN1" (at 55.88 74.93 0)
     (effects (font (size 1.2446 1.2446)) (justify left bottom))
   )
