File: extras/kicad/V2/Power/Power.kicad_pcb (KiCad board)
At the start: 2 copper layers, 760.8 x 135.8 mm, 49 parts, among them J1 1X08_NO_SILK, J2 1X08_NO_SILK, J3 1X08_NO_SILK, J4 1X08_NO_SILK, J5 1X08, J6 1X08, J7 1X08, J8 1X08, SW1 SPDT-HIGH-AMP-SWITCHPTH, U1 CONN-TH_XT60, U1 TB6612FNG, U2 TB6612FNG, U8 POLULUMOTORBRACKETPPCB, X1 6, X2 6, X3 6, X4 6

Commit message: Add files via upload
Parts:
- removed C10, C3, C6, C7, C9: 22u, Capacitor_SMD:C_0805_2012Metric
- removed C11, C2, C4, C5, C8: 100n, Capacitor_SMD:C_0603_1608Metric
- removed H1, H2, H3, H4: Hole, MountingHole:MountingHole_4.3mm_M4_DIN965_Pad_TopBottom
- removed the U1 at (-141.6, 54.2)
- removed U2: TB6612FNG, Package_SO:SSOP-24_5.3x8.2mm_P0.65mm
Other:
- board size 760.8 x 135.8 mm -> 176 x 104.1 mm
- board text removed: "-"
- board text removed: "-1"
- board text removed: "-10"
- board text removed: "-11"
- board text removed: "-12"
- board text removed: "-14"
- board text removed: "-2"
- board text removed: "-3"
- board text removed: "-4"
- board text removed: "-5"
- board text removed: "-6"
- board text removed: "-7"
- board text removed: "-8"
- board text removed: "-9"
- board text removed: "1"
- board text removed: "10 Mbps"
- board text removed: "1751280"
- board text removed: "2"
- board text removed: "3"
- board text removed: "4"
- board text removed: "5"
- board text removed: "6"
- board text removed: "Artemis"
- board text removed: "ENC28J60-H"
- board text removed: "ESP32"
- board text removed: "Ethernet"
- board text removed: "FPGA"
- board text removed: "Featherwing"
- board text removed: "Grove"
- board text removed: "I2C"
- board text removed: "IMU"
- board text removed: "J1"
- board text removed: "J2"
- board text removed: "J3"
- board text removed: "J4"
- board text removed: "J5"
- board text removed: "J6"
- board text removed: "J7"
- board text removed: "J8"
- board text removed: "MS1"
- board text removed: "MicroMod"
- board text removed: "Mount holes for: Jetson Nano/ Beaglebone / Pi 4"
- board text removed: "Olimex.com"
- board text removed: "Optional"
- board text removed: "Qwiic"
- board text removed: "RP2040"
- board text removed: "SPI"
- board text removed: "STM32F405"
- board text removed: "SW1"
- board text removed: "Smartcar\nMotor board rev.0\ndesigned by Dimitris Platis\nhttp://plat.is/smartcar"
- board text removed: "Sparkfun.com"
- board text removed: "Teensy"
- board text removed: "U1"
- board text removed: "U4"
- board text removed: "U8"
- board text removed: "UEXT"
- board text removed: "USB-C"
- board text removed: "X1"
- board text removed: "X2"
- board text removed: "X3"
- board text removed: "X4"
- board text removed: "mikroe.com"
- board text removed: "nRF52840"
- board text removed: "pimoroni.com"
- board text removed: "seeed.cc"

Commit message: Add files via upload
Parts:
- removed 1: NANO-ITX_120X120, easyeda:NANO-ITX_120X120
Changed lines of the file:
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@@
       (net 1 "GND"))
-  )
-  (footprint "easyeda:NANO-ITX_120X120" (layer "F.Cu")
-    (at 415.234 98.321 -90)
-    (attr through_hole)
-    (fp_text reference "1" (at -59.436 -120.396 -90) (layer "B.SilkS")
-      (effects (font (size 1.143 1.143) (thickness 0.152)) (justify left mirror))
-    )
-    (fp_text value "NANO-ITX_120X120" (at -75.179 -123.025 90) (layer "B.Fab") hide
-      (effects (font (size 1.143 1.143) (thickness 0.152)) (justify left mirror))
-    )
-    (fp_text user "gge6377" (at 0 0) (layer "Cmts.User")
-      (effects (font (size 1 1) (thickness 0.15)))
-    )
-    (fp_line (start -119.761 -119.761) (end 0.254 -119.761) (layer "Cmts.User") (width 0.254))
-    (fp_line (start -119.761 0.254) (end -119.761 -119.761) (layer "Cmts.User") (width 0.254))
-    (fp_line (start 0.254 -119.761) (end 0.254 0.254) (layer "Cmts.User") (width 0.254))
-    (fp_line (start 0.254 0.254) (end -119.761 0.254) (layer "Cmts.User") (width 0.254))
-    (fp_line (start -119.38 -119.38) (end 0 -119.38) (layer "Edge.Cuts") (width 0.254))
-    (fp_line (start 0 -119.38) (end 0 0) (layer "Edge.Cuts") (width 0.254))
-    (fp_line (start 0 0) (end -119.38 0) (layer "Edge.Cuts") (width 0.254))
-    (fp_line (start -119.38 0) (end -119.38 -119.38) (layer "Edge.Cuts") (width 0.254))
-    (pad "GND" thru_hole circle locked (at -2.496 -2.746 270) (size 7.6 7.6) (drill oval 4 4.005) (layers F&B.Cu *.Paste *.Mask))
-    (pad "P$2" thru_hole circle locked (at -3.006 -116.506 270) (size 7.6 7.6) (drill oval 4 4.005) (layers F&B.Cu *.Paste *.Mask))
-    (pad "P$3" thru_hole circle locked (at -116.506 -2.746 270) (size 7.6 7.6) (drill oval 4 4.005) (layers F&B.Cu *.Paste *.Mask))
-    (pad "P$4" thru_hole circle locked (at -113.396 -86.726 270) (size 7.6 7.6) (drill oval 4 4.005) (layers F&B.Cu *.Paste *.Mask))
-    (pad "P$11" thru_hole circle locked (at 0.504 -2.746 270) (size 1.308 1.308) (drill oval 0.8 0.805) (layers F&B.Cu *.Paste *.Mask))
-    (pad "P$12" thru_hole circle locked (at -5.496 -2.746 270) (size 1.308 1.308) (drill oval 0.8 0.805) (layers F&B.Cu *.Paste *.Mask))
-    (pad "P$13" thru_hole circle locked (at -2.496 -5.746 270) (size 1.308 1.308) (drill oval 0.8 0.805) (layers F&B.Cu *.Paste *.Mask))
-    (pad "P$14" thru_hole circle locked (at -2.496 0.254 270) (size 1.308 1.308) (drill oval 0.8 0.805) (layers F&B.Cu *.Paste *.Mask))
-    (pad "P$15" thru_hole circle locked (at -0.396 -0.646 270) (size 1.308 1.308) (drill oval 0.8 0.805) (layers F&B.Cu *.Paste *.Mask))
-    (pad "P$16" thru_hole circle locked (at -4.596 -0.646 270) (size 1.308 1.308) (drill oval 0.8 0.805) (layers F&B.Cu *.Paste *.Mask))
-    (pad "P$17" thru_hole circle locked (at -4.596 -4.846 270) (size 1.308 1.308) (drill oval 0.8 0.805) (layers F&B.Cu *.Paste *.Mask))
-    (pad "P$18" thru_hole circle locked (at -0.396 -4.846 270) (size 1.308 1.308) (drill oval 0.8 0.805) (layers F&B.Cu *.Paste *.Mask))
-    (pad "P$20" thru_hole circle locked (at -0.006 -116.506 270) (size 1.308 1.308) (drill oval 0.8 0.805) (layers F&B.Cu *.Paste *.Mask))
-    (pad "P$21" thru_hole circle locked (at -6.006 -116.506 270) (size 1.308 1.308) (drill oval 0.8 0.805) (layers F&B.Cu *.Paste *.Mask))
-    (pad "P$22" thru_hole circle locked (at -3.006 -119.506 270) (size 1.308 1.308) (drill oval 0.8 0.805) (layers F&B.Cu *.Paste *.Mask))
-    (pad "P$23" thru_hole circle locked (at -3.006 -113.506 270) (size 1.308 1.308) (drill oval 0.8 0.805) (layers F&B.Cu *.Paste *.Mask))
-    (pad "P$24" thru_hole circle locked (at -0.906 -114.406 270) (size 1.308 1.308) (drill oval 0.8 0.805) (layers F&B.Cu *.Paste *.Mask))
-    (pad "P$25" thru_hole circle locked (at -5.106 -114.406 270) (size 1.308 1.308) (drill oval 0.8 0.805) (layers F&B.Cu *.Paste *.Mask))
-    (pad "P$26" thru_hole circle locked (at -5.106 -118.606 270) (size 1.308 1.308) (drill oval 0.8 0.805) (layers F&B.Cu *.Paste *.Mask))
-    (pad "P$27" thru_hole circle locked (at -0.906 -118.606 270) (size 1.308 1.308) (drill oval 0.8 0.805) (layers F&B.Cu *.Paste *.Mask))
-    (pad "P$29" thru_hole circle locked (at -113.506 -2.746 270) (size 1.308 1.308) (drill oval 0.8 0.805) (layers F&B.Cu *.Paste *.Mask))
-    (pad "P$30" thru_hole circle locked (at -119.506 -2.746 270) (size 1.308 1.308) (drill oval 0.8 0.805) (layers F&B.Cu *.Paste *.Mask))
-    (pad "P$31" thru_hole circle locked (at -116.506 -5.746 270) (size 1.308 1.308) (drill oval 0.8 0.805) (layers F&B.Cu *.Paste *.Mask))
-    (pad "P$32" thru_hole circle locked (at -116.506 0.254 270) (size 1.308 1.308) (drill oval 0.8 0.805) (layers F&B.Cu *.Paste *.Mask))
-    (pad "P$33" thru_hole circle locked (at -114.406 -0.646 270) (size 1.308 1.308) (drill oval 0.8 0.805) (layers F&B.Cu *.Paste *.Mask))
-    (pad "P$34" thru_hole circle locked (at -118.606 -0.646 270) (size 1.308 1.308) (drill oval 0.8 0.805) (layers F&B.Cu *.Paste *.Mask))
-    (pad "P$35" thru_hole circle locked (at -118.606 -4.846 270) (size 1.308 1.308) (drill oval 0.8 0.805) (layers F&B.Cu *.Paste *.Mask))
-    (pad "P$36" thru_hole circle locked (at -114.406 -4.846 270) (size 1.308 1.308) (drill oval 0.8 0.805) (layers F&B.Cu *.Paste *.Mask))
-    (pad "P$38" thru_hole circle locked (at -110.396 -86.726 270) (size 1.308 1.308) (drill oval 0.8 0.805) (layers F&B.Cu *.Paste *.Mask))
-    (pad "P$39" thru_hole circle locked (at -116.396 -86.726 270) (size 1.308 1.308) (drill oval 0.8 0.805) (layers F&B.Cu *.Paste *.Mask))
-    (pad "P$40" thru_hole circle locked (at -113.396 -89.726 270) (size 1.308 1.308) (drill oval 0.8 0.805) (layers F&B.Cu *.Paste *.Mask))
-    (pad "P$41" thru_hole circle locked (at -113.396 -83.726 270) (size 1.308 1.308) (drill oval 0.8 0.805) (layers F&B.Cu *.Paste *.Mask))
-    (pad "P$42" thru_hole circle locked (at -111.296 -84.626 270) (size 1.308 1.308) (drill oval 0.8 0.805) (layers F&B.Cu *.Paste *.Mask))
-    (pad "P$43" thru_hole circle locked (at -115.496 -84.626 270) (size 1.308 1.308) (drill oval 0.8 0.805) (layers F&B.Cu *.Paste *.Mask))
-    (pad "P$44" thru_hole circle locked (at -115.496 -88.826 270) (size 1.308 1.308) (drill oval 0.8 0.805) (layers F&B.Cu *.Paste *.Mask))
-    (pad "P$45" thru_hole circle locked (at -111.296 -88.826 270) (size 1.308 1.308) (drill oval 0.8 0.805) (layers F&B.Cu *.Paste *.Mask))
   )
   (footprint "easyeda:1X08_NO_SILK" (layer "F.Cu")

Commit message: g
Parts:
- removed ? (x8): , AutoGenerated:MountingHole_3.20mm
- removed J6, J7, J8: 1X08, easyeda:1X08
- removed LOGO1, LOGO2: OSHW-LOGOL, easyeda:OSHW-LOGO-L
- removed MOTOR2, MOTOR3, MOTOR4, MOTOR5: SMARTCAR_MOTOR, easyeda:SMARTCAR_MOTOR_MOUNT_HOLES
- removed SMRTCR1: SMARTCAR_LOGOMEDIUM, easyeda:SMARTCAR_LOGO_MEDIUM
- removed SW1: SPDT-HIGH-AMP-SWITCHPTH, easyeda:SPDT-0.2-THICK-PINS
- removed U$1, U$2: BUMPER_020522_SCREWS, easyeda:BUMPER_2_SCREWS_NARROW
- removed U8: POLULUMOTORBRACKETPPCB, easyeda:POLULUMOTORBRACKETPPCB
- removed X1, X2, X3, X4: 6, easyeda:1751280
- added C10: 22u, Capacitor_SMD:C_0805_2012Metric, F.Cu at (-111.6, 40.6)
- added C11: 100n, Capacitor_SMD:C_0603_1608Metric, F.Cu at (-144.9, 60.5)
- added C2: 100n, Capacitor_SMD:C_0603_1608Metric, F.Cu at (-111.8, 43.4)
- added C3: 22u, Capacitor_SMD:C_0805_2012Metric, F.Cu at (-129.7, 58.8)
- added C4: 100n, Capacitor_SMD:C_0603_1608Metric, F.Cu at (-116.2, 46.4)
- added C5: 100n, Capacitor_SMD:C_0603_1608Metric, F.Cu at (-140.9, 60.5)
- added C6: 22u, Capacitor_SMD:C_0805_2012Metric, F.Cu at (-134.1, 58.8)
- added C7: 22u, Capacitor_SMD:C_0805_2012Metric, F.Cu at (-116.0, 40.6)
- added C8: 100n, Capacitor_SMD:C_0603_1608Metric, F.Cu at (-116.2, 48.9)
- added C9: 22u, Capacitor_SMD:C_0805_2012Metric, F.Cu at (-116.0, 43.7)
- added H1: Hole, MountingHole:MountingHole_4.3mm_M4_DIN965_Pad_TopBottom, F.Cu at (-169.2, 116.7)
- added H2: Hole, MountingHole:MountingHole_4.3mm_M4_DIN965_Pad_TopBottom, F.Cu at (-169.0, 2.65)
- added H3: Hole, MountingHole:MountingHole_4.3mm_M4_DIN965_Pad_TopBottom, F.Cu at (-85.0, 5.75)
- added H4: Hole, MountingHole:MountingHole_4.3mm_M4_DIN965_Pad_TopBottom, F.Cu at (-55.1, 116.2)
- added U1: TB6612FNG, Package_SO:SSOP-24_5.3x8.2mm_P0.65mm, F.Cu at (-141.6, 54.2)
- added U2: TB6612FNG, Package_SO:SSOP-24_5.3x8.2mm_P0.65mm, F.Cu at (-141.6, 44.2)
- added U3: TPS5430DDAR, Package_SO:SOIC-8-1EP_3.9x4.9mm_P1.27mm_EP2.29x3mm_ThermalVias, F.Cu at (-122.0, 87.6)
- U1: value CONN-TH_XT60 -> TB6612FNG; footprint easyeda:CONN-TH_XT60 -> Package_SO:SSOP-24_5.3x8.2mm_P0.65mm
- moved J2 159.1 mm to (541.1, -10.2), turned to -90 degrees
- moved U1 143.2 mm to (402.5, 26.8), turned to 180 degrees
- moved J4 143.0 mm to (414.7, -7.64), turned to -90 degrees
- moved J1 136.5 mm to (541.1, 44.4), turned to -90 degrees
- moved J3 119.9 mm to (414.7, 41.9), turned to -90 degrees
- moved J5 36.6 mm to (486.1, 18.8), turned to 90 degrees
Connections:
- U1 pad 1: (no net) -> Net-(J2-Pad1)
- U1 pad 2: (no net) -> Net-(J2-Pad1)
Other:
- board size 176 x 104.1 mm -> 769.5 x 148.7 mm
- board text added: "1"
- board text added: "1751280"
- board text added: "2"
- board text added: "3"
- board text added: "4"
- board text added: "5"
- board text added: "6"
- board text added: "J1"
- board text added: "J2"
- board text added: "J3"
- board text added: "J4"
- board text added: "J5"
- board text added: "J6"
- board text added: "J7"
- board text added: "J8"
- board text added: "SW1"
- board text added: "Smartcar\nMotor board rev.0\ndesigned by Dimitris Platis\nhttp://plat.is/smartcar"
- board text added: "U1"
- board text added: "U8"
- board text added: "X1"
- board text added: "X2"
- board text added: "X3"
- board text added: "X4"

Commit message: g
Parts:
- removed the U1 at (-141.6, 54.2)
- removed the U1 at (402.5, 26.8)
- added C12: 100n, Capacitor_SMD:C_0603_1608Metric, F.Cu at (267.8, 78.0)
- added C13: 22u, Capacitor_SMD:C_0805_2012Metric, F.Cu at (247.5, 85.3)
- added C14: 100n, Capacitor_SMD:C_0603_1608Metric, F.Cu at (268.3, 73.0)
- added C15: 22u, Capacitor_SMD:C_0805_2012Metric, F.Cu at (251.1, 79.2)
- added C19: 22u, Capacitor_SMD:C_0805_2012Metric, F.Cu at (243.1, 82.3)
- added C20: 22u, Capacitor_SMD:C_0805_2012Metric, F.Cu at (243.1, 88.3)
- added C21: 100n, Capacitor_SMD:C_0603_1608Metric, F.Cu at (259.8, 87.0)
- added C22: 100n, Capacitor_SMD:C_0603_1608Metric, F.Cu at (260.2, 81.5)
- added C23: 22u, Capacitor_SMD:C_0805_2012Metric, F.Cu at (247.5, 88.3)
- added C24: 100n, Capacitor_SMD:C_0603_1608Metric, F.Cu at (255.8, 87.5)
- added C25: 22u, Capacitor_SMD:C_0805_2012Metric, F.Cu at (243.1, 85.3)
- added C26: 22u, Capacitor_SMD:C_0805_2012Metric, F.Cu at (255.6, 76.2)
- added C27: 22u, Capacitor_SMD:C_0805_2012Metric, F.Cu at (247.5, 82.3)
- added C28: 22u, Capacitor_SMD:C_0805_2012Metric, F.Cu at (251.1, 76.2)
- added C29: 100n, Capacitor_SMD:C_0603_1608Metric, F.Cu at (264.2, 75.5)
- added C30: 22u, Capacitor_SMD:C_0805_2012Metric, F.Cu at (251.1, 73.2)
- added D1: D, Diode_SMD:D_SMA, F.Cu at (244.9, 74.0)
- added D2: D, Diode_SMD:D_SMA, F.Cu at (244.9, 78.5)
- added H5: Motor, Z_mycustom_footprint_lib:JGA25-370 DC motor, B.Cu at (70.0, 70.0)
- added H6: Motor, Z_mycustom_footprint_lib:JGA25-370 DC motor, B.Cu at (160.0, 70.0)
- added H7: Motor, Z_mycustom_footprint_lib:JGA25-370 DC motor, B.Cu at (160.0, 140.0)
- added H8: Motor, Z_mycustom_footprint_lib:JGA25-370 DC motor, B.Cu at (70.0, 140.0)
- added J6: Conn_02x20_Odd_Even, Connector_PinHeader_2.54mm:PinHeader_2x20_P2.54mm_Vertical, F.Cu at (90.6, 58.7)
- added J7: Conn_02x20_Odd_Even, Connector_PinHeader_2.54mm:PinHeader_2x20_P2.54mm_Vertical, F.Cu at (91.1, 143.8)
- added R12: 0.1, Resistor_SMD:R_1206_3216Metric_Pad1.30x1.75mm_HandSolder, F.Cu at (46.0, 97.2)
- added R13: 0.1, Resistor_SMD:R_1206_3216Metric_Pad1.30x1.75mm_HandSolder, F.Cu at (46.0, 87.6)
- added R14: 1Meg, Resistor_SMD:R_0603_1608Metric, F.Cu at (263.8, 79.0)
- added R15: 1Meg, Resistor_SMD:R_0603_1608Metric, F.Cu at (264.2, 73.0)
- added R16: 100k, Resistor_SMD:R_0603_1608Metric, F.Cu at (259.8, 84.5)
- added R2: 0.1, Resistor_SMD:R_1206_3216Metric_Pad1.30x1.75mm_HandSolder, F.Cu at (46.0, 90.0)
- added R3: 10k, Resistor_SMD:R_0603_1608Metric, F.Cu at (264.2, 81.5)
- added R4: 100k, Resistor_SMD:R_0603_1608Metric, F.Cu at (256.2, 82.0)
- added R7: 0.1, Resistor_SMD:R_1206_3216Metric_Pad1.30x1.75mm_HandSolder, F.Cu at (46.0, 94.8)
- added R8: 10k, Resistor_SMD:R_0603_1608Metric, F.Cu at (251.8, 85.0)
- added R9: 0.1, Resistor_SMD:R_1206_3216Metric_Pad1.30x1.75mm_HandSolder, F.Cu at (46.0, 92.4)
- added SMRTCR1: SMARTCAR_LOGOMEDIUM, easyeda:SMARTCAR_LOGO_MEDIUM, B.Cu at (116.2, 103.2)
- added U1: TB6612FNG, Package_SO:SSOP-24_5.3x8.2mm_P0.65mm, F.Cu at (127.4, 78.1)
- added U4: TPS5430DDAR, Package_SO:SOIC-8-1EP_3.9x4.9mm_P1.27mm_EP2.29x3mm_ThermalVias, F.Cu at (101.8, 130.4)
- J1: value 1X08_NO_SILK -> Conn_01x02; footprint easyeda:1X08_NO_SILK -> Connector_AMASS:AMASS_XT60-M_1x02_P7.20mm_Vertical
- J2, J3, J4: value 1X08_NO_SILK -> Screw_Terminal_01x06; footprint easyeda:1X08_NO_SILK -> TerminalBlock_4Ucon:TerminalBlock_4Ucon_1x06_P3.50mm_Horizontal; moved to B.Cu
- J5: value 1X08 -> Screw_Terminal_01x06; footprint easyeda:1X08 -> TerminalBlock_4Ucon:TerminalBlock_4Ucon_1x06_P3.50mm_Horizontal; moved to B.Cu
- moved J1 508.6 mm to (36.3, 106.7), turned to 90 degrees
- moved J2 478.1 mm to (78.1, 109.1), turned to 180 degrees
- moved J5 416.0 mm to (78.1, 100.0), turned to 180 degrees
- moved C5 409.4 mm to (268.3, 75.5)
- moved C11 401.4 mm to (255.8, 85.0)
- moved C6 394.4 mm to (260.0, 73.2)
- moved C4 389.4 mm to (272.3, 73.0)
- moved C3 382.4 mm to (252.0, 82.3)
- moved C9 377.5 mm to (260.0, 76.2)
- moved C2 373.3 mm to (259.8, 79.0)
- moved C7 373.0 mm to (255.6, 73.2)
- moved H2 371.9 mm to (192.2, 91.1), turned to 90 degrees
- moved C8 370.0 mm to (251.8, 87.5)
- moved C10 369.2 mm to (255.6, 79.2)
- moved H1 361.4 mm to (192.2, 118.9), turned to 90 degrees
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Connections:
- J1 pad 1: (no net) -> GND
- J1 pad 2: (no net) -> Net-(J1-Pad2)
- J2 pad 1: (no net) -> /Black_1
- J2 pad 2: (no net) -> /Blue_1
- J2 pad 3: (no net) -> /Green_1
- J2 pad 4: (no net) -> /yellow_1
- J2 pad 5: (no net) -> /AO2_1
- J2 pad 6: (no net) -> /AO1_1
- J3 pad 1: (no net) -> /Black_2
- J3 pad 2: (no net) -> /Blue_2
- J3 pad 3: (no net) -> /Green_2
- J3 pad 4: (no net) -> /yellow_2
- J3 pad 5: (no net) -> /BO2_1
- J3 pad 6: (no net) -> /BO1_1
- J4 pad 1: (no net) -> /Black_3
- J4 pad 2: (no net) -> /Blue_3
- J4 pad 3: (no net) -> /Green_3
- J4 pad 4: (no net) -> /yellow_3
- J4 pad 5: (no net) -> /AO2_2
- J4 pad 6: (no net) -> /AO1_2
- J5 pad 1: (no net) -> /Black_4
- J5 pad 2: (no net) -> /Blue_4
- J5 pad 3: GND -> /Green_4
- J5 pad 4: (no net) -> /yellow_4
- J5 pad 5: (no net) -> /BO2_2
- J5 pad 6: (no net) -> /BO1_2
- U2 pad 1: Net-(J3-Pad1) -> /AO1_2
- U2 pad 11: Net-(J5-Pad1) -> /BO1_2
- U2 pad 12: Net-(J5-Pad1) -> /BO1_2
- U2 pad 2: Net-(J3-Pad1) -> /AO1_2
- U2 pad 5: Net-(J3-Pad2) -> /AO2_2
- U2 pad 6: Net-(J3-Pad2) -> /AO2_2
- U2 pad 7: Net-(J5-Pad2) -> /BO2_2
- U2 pad 8: Net-(J5-Pad2) -> /BO2_2
Routing:
- net GND: track 1731.3 -> 0.00 mm, vias 12 -> 0
- net (no net): track 463.7 -> 0.00 mm, vias 1 -> 0
- added copper zone on F.Cu, net GND
Other:
- board size 769.5 x 148.7 mm -> 181.3 x 110 mm
- board text removed: "1"
- board text removed: "1751280"
- board text removed: "2"
- board text removed: "3"
- board text removed: "4"
- board text removed: "5"
- board text removed: "6"
- board text removed: "EN_GND"
- board text removed: "EN_L_1"
- board text removed: "EN_L_2"
- board text removed: "EN_R_1"
- board text removed: "EN_R_2"
- board text removed: "EN_VCC"
- board text removed: "GND"
- board text removed: "J1"
- board text removed: "J2"
- board text removed: "J3"
- board text removed: "J4"
- board text removed: "J5"
- board text removed: "J6"
- board text removed: "J7"
- board text removed: "J8"
- board text removed: "MOTOR_L_OUT1"
- board text removed: "MOTOR_L_OUT2"
- board text removed: "MOTOR_R_OUT1"
- board text removed: "MOTOR_R_OUT2"
- board text removed: "OFF"
- board text removed: "ON"
- board text removed: "SW1"
- board text removed: "Smartcar Motor board rev.0 designed by Dimitris Platis http://plat.is/smartcar"
- board text removed: "Smartcar\nMotor board rev.0\ndesigned by Dimitris Platis\nhttp://plat.is/smartcar"
- board text removed: "TB6612FNG"
- board text removed: "U1"
- board text removed: "U8"
- board text removed: "V MOTOR"
- board text removed: "VCC_EN"
- board text removed: "X1"
- board text removed: "X2"
- board text removed: "X3"
- board text removed: "X4"

Commit message: f
Parts:
- removed SMRTCR1: SMARTCAR_LOGOMEDIUM, easyeda:SMARTCAR_LOGO_MEDIUM
- added C16: 4n7, Capacitor_SMD:C_0603_1608Metric_Pad1.08x0.95mm_HandSolder, F.Cu at (102.6, 80.3)
- added C17: 10n, Capacitor_SMD:C_0603_1608Metric_Pad1.08x0.95mm_HandSolder, F.Cu at (100.0, 77.6)
- added C18: 39p, Capacitor_SMD:C_0603_1608Metric_Pad1.08x0.95mm_HandSolder, F.Cu at (105.1, 79.5)
- added C31: 10n, Capacitor_SMD:C_0603_1608Metric_Pad1.08x0.95mm_HandSolder, F.Cu at (251.6, 101.2)
- added C32: 47p, Capacitor_SMD:C_0603_1608Metric_Pad1.08x0.95mm_HandSolder, F.Cu at (255.9, 98.7)
- added C33: 1n, Capacitor_SMD:C_0603_1608Metric_Pad1.08x0.95mm_HandSolder, F.Cu at (247.2, 103.7)
- added L1: 6u8, Z_mycustom_footprint_lib:Inductor SMD,11.6x10.1x4mm, F.Cu at (114.3, 77.7)
- added L2: 6u8, Z_mycustom_footprint_lib:Inductor SMD,11.6x10.1x4mm, F.Cu at (255.2, 48.8)
- added R10: 3k24, Resistor_SMD:R_0603_1608Metric_Pad0.98x0.95mm_HandSolder, F.Cu at (240.7, 56.1)
- added R11: 29.4, Capacitor_SMD:C_0603_1608Metric_Pad1.08x0.95mm_HandSolder, F.Cu at (251.6, 103.7)
- added R5: 1k91, Resistor_SMD:R_0603_1608Metric_Pad0.98x0.95mm_HandSolder, F.Cu at (106.9, 77.9)
- added R6: 49.9, Capacitor_SMD:C_0603_1608Metric_Pad1.08x0.95mm_HandSolder, F.Cu at (105.1, 81.1)
- moved C14 168.3 mm to (100.0, 72.9), turned to 90 degrees
- moved C12 166.6 mm to (101.4, 69.8), turned to 90 degrees
- moved R14 165.5 mm to (98.4, 74.5), turned to -90 degrees
- moved R4 158.7 mm to (97.6, 76.7), turned to 180 degrees
- moved R3 156.4 mm to (107.8, 80.3), turned to 90 degrees
- moved H3 153.9 mm to (45.0, 65.0)
- moved H4 153.7 mm to (45.0, 145.0)
- moved C13 151.3 mm to (96.6, 74.2), turned to -90 degrees
- moved D1 139.0 mm to (105.9, 69.3), turned to 180 degrees
- moved U1 31.4 mm to (128.5, 109.5)
- moved H1 27.1 mm to (185.0, 145.0)
- moved H2 27.1 mm to (185.0, 65.0)
- moved U2 22.2 mm to (116.2, 108.6)
- moved U3 13.2 mm to (104.6, 74.3)
- moved J7 6.23 mm to (91.0, 150.0)
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Connections:
- net Net-(R10-Pad1) renamed /3v3_FB
- net Net-(R4-Pad1) renamed /EN1
- net Net-(R5-Pad1) renamed /5v_FB
- net Net-(U4-Pad3) renamed /EN2
- U3 pad 4: Net-(C17-Pad1) -> /ss1
- U4 pad 4: Net-(C31-Pad1) -> /ss2
Routing:
- net Net-(C12-Pad2): track 0.00 -> 20.3 mm
- net GND: track 0.00 -> 13.6 mm, vias 0 -> 2
- net Net-(C16-Pad2): track 0.00 -> 10.6 mm, vias 0 -> 2
- net +12V: track 0.00 -> 8.33 mm
- net +5V: track 0.00 -> 7.06 mm
- net /EN1: track 0.00 -> 5.03 mm
- net /5v_FB: track 0.00 -> 3.56 mm
- net /ss1: track 0.00 -> 2.36 mm
- net Net-(C12-Pad1): track 0.00 -> 2.12 mm
- net Net-(C16-Pad1): track 0.00 -> 1.66 mm

Commit message: t
Parts:
- moved R15 180.6 mm to (92.5, 128.9), turned to -90 degrees
- moved R16 172.0 mm to (94.1, 130.6), turned to -90 degrees
- moved L2 169.0 mm to (108.2, 132.2), turned to -90 degrees
- moved C24 166.5 mm to (94.1, 127.2), turned to 90 degrees
- moved C23 162.0 mm to (90.7, 129.0), turned to -90 degrees
- moved C32 161.5 mm to (98.7, 135.5)
- moved R10 159.7 mm to (100.4, 132.3), turned to 180 degrees
- moved R8 158.4 mm to (101.3, 134.6), turned to 90 degrees
- moved C31 157.6 mm to (97.0, 132.3)
- moved R11 155.8 mm to (98.7, 133.9)
- moved C33 154.2 mm to (96.2, 134.8), turned to -90 degrees
- moved D2 150.5 mm to (101.4, 124.1), turned to 180 degrees
- moved C21 139.6 mm to (120.2, 87.0), turned to -90 degrees
- moved C15 137.1 mm to (114.2, 87.1), turned to -90 degrees
- moved C19 126.9 mm to (116.3, 87.1), turned to -90 degrees
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Connections:
- net Net-(C12-Pad2) renamed /SW1
- net Net-(C22-Pad2) renamed /SW2
Routing:
- net +12V: track 8.33 -> 77.0 mm
- net +5V: track 7.06 -> 29.7 mm
- net Net-(J1-Pad2): track 0.00 -> 18.7 mm
- net GND: track 13.6 -> 26.6 mm, vias 2 -> 17
- added copper zone on F.Cu, net +5V
- added copper zone on F.Cu, net /SW1
