File: extras/kicad/V2/Power/Power.kicad_pcb (KiCad board)
At the start: 2 copper layers, 181.3 x 110 mm, 70 parts, among them J1 Conn_01x02, J2 Screw_Terminal_01x06, J3 Screw_Terminal_01x06, J4 Screw_Terminal_01x06, J5 Screw_Terminal_01x06, J6 Conn_02x20_Odd_Even, J7 Conn_02x20_Odd_Even, U1 TB6612FNG, U2 TB6612FNG, U3 TPS5430DDAR, U4 TPS5430DDAR

Commit message: n
Parts:
- removed R10: 3k24, Resistor_SMD:R_0603_1608Metric_Pad0.98x0.95mm_HandSolder
- removed R11: 29.4, Capacitor_SMD:C_0603_1608Metric_Pad1.08x0.95mm_HandSolder
- removed R14, R15: 1Meg, Resistor_SMD:R_0603_1608Metric
- removed R16: 100k, Resistor_SMD:R_0603_1608Metric
- removed R8: 10k, Resistor_SMD:R_0603_1608Metric
- added C1: 1n5, Capacitor_SMD:C_0603_1608Metric_Pad1.08x0.95mm_HandSolder, F.Cu at (234.6, 116.8)
- added C34: 100n, Capacitor_SMD:C_0603_1608Metric, F.Cu at (114.0, 67.6)
- added TP1: TestPoint, TestPoint:TestPoint_Pad_D1.0mm, F.Cu at (238.0, 120.1)
- added TP2: TestPoint, TestPoint:TestPoint_Pad_D1.0mm, F.Cu at (238.3, 117.1)
- C13, C15, C19, C20, C27, C28, C30: value 22u -> 47u; footprint Capacitor_SMD:C_0805_2012Metric -> Capacitor_SMD:C_1206_3216Metric
- C16: value 4n7 -> 1n5
- C17, C31: value 10n -> 47u; footprint Capacitor_SMD:C_0603_1608Metric_Pad1.08x0.95mm_HandSolder -> Capacitor_SMD:C_1206_3216Metric
- C18: value 39p -> 47u; footprint Capacitor_SMD:C_0603_1608Metric_Pad1.08x0.95mm_HandSolder -> Capacitor_SMD:C_1206_3216Metric
- C22, C24, C29: value 100n -> 47u; footprint Capacitor_SMD:C_0603_1608Metric -> Capacitor_SMD:C_1206_3216Metric
- C23, C25: value 22u -> 100n; footprint Capacitor_SMD:C_0805_2012Metric -> Capacitor_SMD:C_0603_1608Metric
- C26: value 22u -> 1n5; footprint Capacitor_SMD:C_0805_2012Metric -> Capacitor_SMD:C_0603_1608Metric_Pad1.08x0.95mm_HandSolder
- C32: value 47p -> 47u; footprint Capacitor_SMD:C_0603_1608Metric_Pad1.08x0.95mm_HandSolder -> Capacitor_SMD:C_1206_3216Metric
- C33: value 1n -> 47u; footprint Capacitor_SMD:C_0603_1608Metric_Pad1.08x0.95mm_HandSolder -> Capacitor_SMD:C_1206_3216Metric
- L1, L2: value 6u8 -> 15u
- R4: value 100k -> 10k
- R5: value 1k91 -> 3k24
- R6: value 49.9 -> 5k9; footprint Capacitor_SMD:C_0603_1608Metric_Pad1.08x0.95mm_HandSolder -> Resistor_SMD:R_0603_1608Metric_Pad0.98x0.95mm_HandSolder
- moved C14 191.5 mm to (280.7, 136.4), turned to 0 degrees
- moved C12 191.4 mm to (282.6, 131.4), turned to 0 degrees
- moved C13 190.4 mm to (279.1, 128.5), turned to 0 degrees
- moved C17 180.7 mm to (270.2, 138.3), turned to 0 degrees
- moved C18 180.6 mm to (275.9, 138.3)
- moved R5 179.7 mm to (278.4, 131.4), turned to 0 degrees
- moved R3 178.0 mm to (275.1, 141.2), turned to 0 degrees
- moved U3 176.4 mm to (272.0, 130.0)
- moved C16 173.7 mm to (261.5, 150.3), turned to 0 degrees
- moved C20 171.4 mm to (284.7, 128.5), turned to 0 degrees
- moved D1 170.8 mm to (263.4, 135.5), turned to 0 degrees
- moved C19 161.2 mm to (270.2, 134.9), turned to 0 degrees
- moved C21 158.9 mm to (267.0, 147.9), turned to 0 degrees
- moved C15 158.5 mm to (262.2, 144.0), turned to 0 degrees
- moved C29 154.6 mm to (109.8, 69.6), turned to 180 degrees
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Connections:
- C12 pad 2: /SW1 -> Net-(C12-Pad2)
- C16 pad 1: Net-(C16-Pad1) -> +5V
- C16 pad 2: Net-(C16-Pad2) -> /5v_FB
- C17 pad 1: /ss1 -> +5V
- C18 pad 1: Net-(C16-Pad2) -> +5V
- C22 pad 1: Net-(C22-Pad1) -> +5V
- C22 pad 2: /SW2 -> GND
- C23 pad 1: +12V -> Net-(C23-Pad1)
- C23 pad 2: GND -> Net-(C23-Pad2)
- C25 pad 1: +3V3 -> +12V
- C26 pad 2: GND -> /3v3_FB
- C31 pad 1: /ss2 -> +3V3
- C32 pad 1: Net-(C32-Pad1) -> +3V3
- C33 pad 1: Net-(C33-Pad1) -> +3V3
- C33 pad 2: Net-(C32-Pad1) -> GND
- D1 pad 1: /SW1 -> Net-(C12-Pad1)
- D2 pad 1: /SW2 -> Net-(C23-Pad1)
- L1 pad 1: /SW1 -> Net-(C12-Pad1)
- L2 pad 1: /SW2 -> Net-(C23-Pad1)
- R4 pad 1: /EN1 -> +3V3
- R4 pad 2: GND -> /3v3_FB
- R6 pad 1: Net-(C16-Pad1) -> /3v3_FB
- U3 pad 1: Net-(C12-Pad1) -> Net-(C12-Pad2)
- U3 pad 2: +12V -> unconnected-(U3-Pad2)
- U3 pad 3: /EN1 -> unconnected-(U3-Pad3)
- U3 pad 4: /ss1 -> /5v_FB
- U3 pad 5: /5v_FB -> Net-(U3-Pad5)
- U3 pad 6: Net-(C16-Pad2) -> GND
- U3 pad 7: GND -> +12V
- U3 pad 8: /SW1 -> Net-(C12-Pad1)
- U4 pad 1: Net-(C22-Pad1) -> Net-(C23-Pad2)
- U4 pad 2: +12V -> unconnected-(U4-Pad2)
- U4 pad 3: /EN2 -> unconnected-(U4-Pad3)
- U4 pad 4: /ss2 -> /3v3_FB
- U4 pad 5: /3v3_FB -> Net-(TP2-Pad1)
- U4 pad 6: Net-(C32-Pad1) -> GND
- U4 pad 7: GND -> +12V
- U4 pad 8: /SW2 -> Net-(C23-Pad1)
Routing:
- net +3V3: track 0.00 -> 38.4 mm, vias 0 -> 2
- net +5V: track 29.7 -> 0.00 mm
- net /SW1: track 20.6 -> 0.00 mm
- net Net-(C23-Pad1): track 0.00 -> 19.8 mm
- net Net-(C16-Pad2): track 10.7 -> 0.00 mm, vias 2 -> 0
- net +12V: track 77.0 -> 66.5 mm
- net GND: track 26.6 -> 17.2 mm, vias 17 -> 31
- net /EN1: track 5.27 -> 0.00 mm
- net /3v3_FB: track 0.00 -> 5.02 mm
- net /5v_FB: track 3.55 -> 0.00 mm
- net /ss1: track 2.36 -> 0.00 mm
- net Net-(C12-Pad1): track 2.12 -> 0.00 mm
- net Net-(C23-Pad2): track 0.00 -> 1.83 mm
- net Net-(C16-Pad1): track 1.66 -> 0.00 mm
- added copper zone on F.Cu, net +3V3
- removed copper zone on F.Cu, net +5V
- removed copper zone on F.Cu, net /SW1

Commit message: g
Parts:
- moved C20 187.6 mm to (97.3, 136.6), turned to 180 degrees
- moved C12 176.5 mm to (106.4, 121.4), turned to -90 degrees
- moved C18 173.8 mm to (102.1, 136.6)
- moved C17 172.9 mm to (97.3, 139.0), turned to 180 degrees
- moved R5 171.2 mm to (107.2, 129.4)
- moved C22 171.2 mm to (97.3, 134.2), turned to 180 degrees
- moved R3 169.0 mm to (106.3, 132.0), turned to 90 degrees
- moved C19 168.1 mm to (102.1, 139.0)
- moved C14 167.5 mm to (113.6, 125.9), turned to -90 degrees
- moved C21 164.9 mm to (102.2, 141.0)
- moved C13 163.5 mm to (115.6, 126.1), turned to -90 degrees
- moved U3 163.1 mm to (109.0, 125.8)
- moved C15 160.4 mm to (102.1, 134.2)
- moved C16 154.7 mm to (107.9, 132.0), turned to 90 degrees
- moved D1 153.0 mm to (111.1, 121.2), turned to 180 degrees
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Routing:
- net Net-(C12-Pad1): track 0.00 -> 23.2 mm
- net +5V: track 0.00 -> 15.0 mm, vias 0 -> 2
- net GND: track 17.2 -> 28.2 mm, vias 31 -> 65
- net /5v_FB: track 0.00 -> 5.18 mm
- net +12V: track 66.5 -> 70.8 mm
- net Net-(TP2-Pad1): track 0.00 -> 1.99 mm
- net Net-(U3-Pad5): track 0.00 -> 1.91 mm
- net Net-(C12-Pad2): track 0.00 -> 1.77 mm
- added copper zone on F.Cu, net +5V
