File: extras/kicad/V2/Power/Power.kicad_pcb (KiCad board)
At the start: 2 copper layers, 181.3 x 110 mm, 68 parts, among them J1 Conn_01x02, J2 Screw_Terminal_01x06, J3 Screw_Terminal_01x06, J4 Screw_Terminal_01x06, J5 Screw_Terminal_01x06, J6 Conn_02x20_Odd_Even, J7 Conn_02x20_Odd_Even, U1 TB6612FNG, U2 TB6612FNG, U3 TPS5430DDAR, U4 TPS5430DDAR

Commit message: g
Parts:
- added H10: Bumper, MountingHole:MountingHole_4.5mm, F.Cu at (34.5, 125.6)
- added H11: Bumper, MountingHole:MountingHole_4.5mm, F.Cu at (195.8, 87.4)
- added H12: Bumper, MountingHole:MountingHole_4.5mm, F.Cu at (34.5, 86.6)
- added H9: Bumper, MountingHole:MountingHole_4.5mm, F.Cu at (195.8, 126.4)
- C10, C11, C12, C13, C14, C15, C16, C17, C18, C19, C20, C21, C22, C23, C24, C25, C26, C27, C28, C29, C3, C30, C31, C32, C33, C34, C4, C5, C6, C7, C8, C9, D1, D2, L1, L2, R12, R13, R2, R3, R4, R5, R6, R7, R9, TP1, TP2, U1, U2, U3, U4: moved to B.Cu
- moved C3 196.3 mm to (58.0, 99.5), turned to -90 degrees
- moved C10 147.4 mm to (111.6, 107.5), turned to -90 degrees
- moved C8 146.5 mm to (115.4, 90.1), turned to 180 degrees
- moved C4 145.4 mm to (117.6, 106.9)
- moved C5 139.3 mm to (118.7, 90.1), turned to 180 degrees
- moved C9 139.1 mm to (109.5, 107.5), turned to -90 degrees
- moved C7 132.6 mm to (121.9, 90.3), turned to 180 degrees
- moved C11 130.9 mm to (122.0, 106.9)
- moved C6 127.4 mm to (121.9, 92.4), turned to 180 degrees
- moved J2 68.9 mm to (137.4, 74.2)
- moved J5 68.2 mm to (134.2, 138.9)
- moved J3 51.7 mm to (131.2, 65.8)
- moved J4 36.8 mm to (138.2, 130.5)
- moved U1 26.6 mm to (119.8, 84.4), turned to -90 degrees
- moved C13 24.7 mm to (91.0, 128.4)
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Connections:
- J2 pad 5: /AO2_1 -> /BO1_1
- J2 pad 6: /AO1_1 -> /BO2_1
- J3 pad 5: /BO2_1 -> /AO2_1
- J3 pad 6: /BO1_1 -> /AO1_1
- J4 pad 5: /AO2_2 -> /AO1_2
- J4 pad 6: /AO1_2 -> /AO2_2
- J6 pad 10: unconnected-(J6-Pad10) -> GND
- J6 pad 25: unconnected-(J6-Pad25) -> /yellow_2
- J6 pad 26: unconnected-(J6-Pad26) -> GND
- J6 pad 27: unconnected-(J6-Pad27) -> /Green_2
- J6 pad 29: unconnected-(J6-Pad29) -> /Blue_2
- J6 pad 3: unconnected-(J6-Pad3) -> GND
- J6 pad 31: unconnected-(J6-Pad31) -> /Black_2
- J6 pad 32: unconnected-(J6-Pad32) -> GND
- J6 pad 33: unconnected-(J6-Pad33) -> /yellow_1
- J6 pad 35: unconnected-(J6-Pad35) -> /Green_1
- J6 pad 37: unconnected-(J6-Pad37) -> /Blue_1
- J6 pad 38: unconnected-(J6-Pad38) -> GND
- J6 pad 39: unconnected-(J6-Pad39) -> /Black_1
- J6 pad 4: unconnected-(J6-Pad4) -> GND
- J6 pad 5: unconnected-(J6-Pad5) -> +3V3
- J6 pad 6: unconnected-(J6-Pad6) -> +3V3
- J6 pad 7: unconnected-(J6-Pad7) -> +3V3
- J6 pad 8: unconnected-(J6-Pad8) -> +3V3
- J6 pad 9: unconnected-(J6-Pad9) -> GND
- J7 pad 11: unconnected-(J7-Pad11) -> GND
- J7 pad 12: unconnected-(J7-Pad12) -> GND
- J7 pad 13: unconnected-(J7-Pad13) -> +5V
- J7 pad 14: unconnected-(J7-Pad14) -> +5V
- J7 pad 15: unconnected-(J7-Pad15) -> +5V
- J7 pad 16: unconnected-(J7-Pad16) -> +5V
- J7 pad 17: unconnected-(J7-Pad17) -> GND
- J7 pad 18: unconnected-(J7-Pad18) -> GND
- J7 pad 25: unconnected-(J7-Pad25) -> GND
- J7 pad 26: unconnected-(J7-Pad26) -> /yellow_4
- J7 pad 28: unconnected-(J7-Pad28) -> /Green_4
- J7 pad 30: unconnected-(J7-Pad30) -> /Blue_4
- J7 pad 31: unconnected-(J7-Pad31) -> GND
- J7 pad 32: unconnected-(J7-Pad32) -> /Black_4
- J7 pad 34: unconnected-(J7-Pad34) -> /yellow_3
- J7 pad 36: unconnected-(J7-Pad36) -> /Green_3
- J7 pad 37: unconnected-(J7-Pad37) -> GND
- J7 pad 38: unconnected-(J7-Pad38) -> /Blue_3
- J7 pad 40: unconnected-(J7-Pad40) -> /Black_3
Routing:
- net +12V: track 70.8 -> 240.4 mm
- net +5V: track 15.0 -> 117.3 mm, vias 2 -> 5
- net GND: track 28.2 -> 82.5 mm, vias 65 -> 100
- net +3V3: track 38.4 -> 64.4 mm
- net /yellow_3: track 0.00 -> 25.8 mm
- net /BO2_2: track 0.00 -> 24.7 mm
- net /BO1_2: track 0.00 -> 23.8 mm
- net /Green_3: track 0.00 -> 23.4 mm
- net /Blue_3: track 0.00 -> 22.1 mm
- net /yellow_1: track 0.00 -> 22.1 mm
- net /Black_3: track 0.00 -> 19.9 mm
- net /Green_1: track 0.00 -> 19.5 mm
- net /Blue_1: track 0.00 -> 18.3 mm
- net /Black_1: track 0.00 -> 17.9 mm
- net /AO2_1: track 0.00 -> 16.2 mm
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- added copper zone on B.Cu, net +3V3
- added copper zone on B.Cu, net +5V
- removed copper zone on F.Cu, net +3V3
- removed copper zone on F.Cu, net +5V

Commit message: g
Connections:
- J7 pad 10: unconnected-(J7-Pad10) -> PWMA_2
- J7 pad 2: unconnected-(J7-Pad2) -> PWMB_2
- J7 pad 3: unconnected-(J7-Pad3) -> GND
- J7 pad 4: unconnected-(J7-Pad4) -> BIN2_2
- J7 pad 5: unconnected-(J7-Pad5) -> BIN1_2
- J7 pad 6: unconnected-(J7-Pad6) -> GND
- J7 pad 7: unconnected-(J7-Pad7) -> STBY_2
- J7 pad 8: unconnected-(J7-Pad8) -> AIN1_2
- J7 pad 9: unconnected-(J7-Pad9) -> AIN2_2
Routing:
- net AIN2_2: track 0.00 -> 80.7 mm
- net STBY_2: track 0.00 -> 78.5 mm
- net PWMA_2: track 0.00 -> 78.1 mm
- net AIN1_2: track 0.00 -> 76.6 mm
- net BIN1_2: track 0.00 -> 75.6 mm
- net BIN2_2: track 0.00 -> 72.0 mm
- net PWMB_2: track 0.00 -> 71.0 mm
- net +12V: track 240.4 -> 230.7 mm, vias 0 -> 10
- added copper zone on F.Cu, net +12V

Commit message: n
Parts:
- added TP3: TestPoint, TestPoint:TestPoint_Pad_D1.0mm, B.Cu at (52.7, 115.9)
- added TP4: TestPoint, TestPoint:TestPoint_Pad_D1.0mm, B.Cu at (55.9, 115.9)
- added TP5: TestPoint, TestPoint:TestPoint_Pad_D1.0mm, B.Cu at (52.9, 91.6)
- added TP6: TestPoint, TestPoint:TestPoint_Pad_D1.0mm, B.Cu at (55.0, 91.5)
- added U5: INA219AxD, Package_SO:SOIC-8_3.9x4.9mm_P1.27mm, B.Cu at (55.6, 96.6)
- C1: value 1n5 -> 100n; footprint Capacitor_SMD:C_0603_1608Metric_Pad1.08x0.95mm_HandSolder -> Capacitor_SMD:C_0603_1608Metric; moved to B.Cu
- C2: moved to B.Cu
- J6: value Conn_02x20_Odd_Even -> left
- J7: value Conn_02x20_Odd_Even -> right
- moved C2 209.4 mm to (58.0, 101.3)
- moved C1 204.4 mm to (54.3, 101.3), turned to 180 degrees
- moved J4 17.8 mm to (120.4, 130.5), turned to 0 degrees
- moved J3 17.5 mm to (113.8, 65.9), turned to 0 degrees
- moved R12 11.9 mm to (54.2, 105.6)
- moved R7 11.8 mm to (54.2, 107.9)
- moved R9 11.7 mm to (54.2, 110.2)
- moved R2 11.7 mm to (54.2, 112.6)
- moved C3 7.91 mm to (58.4, 107.4)
Connections:
- C1 pad 1: unconnected-(C1-Pad1) -> +12V
- C1 pad 2: unconnected-(C1-Pad2) -> Net-(J1-Pad2)
- C2 pad 1: unconnected-(C2-Pad1) -> GND
- C2 pad 2: unconnected-(C2-Pad2) -> +5V
- J3 pad 1: /Black_2 -> /AO1_1
- J3 pad 2: /Blue_2 -> /AO2_1
- J3 pad 3: /Green_2 -> /yellow_2
- J3 pad 4: /yellow_2 -> /Green_2
- J3 pad 5: /AO2_1 -> /Blue_2
- J3 pad 6: /AO1_1 -> /Black_2
- J4 pad 1: /Black_3 -> /AO2_2
- J4 pad 2: /Blue_3 -> /AO1_2
- J4 pad 3: /Green_3 -> /yellow_3
- J4 pad 4: /yellow_3 -> /Green_3
- J4 pad 5: /AO1_2 -> /Blue_3
- J4 pad 6: /AO2_2 -> /Black_3
- J6 pad 1: unconnected-(J6-Pad1) -> SCL
- J6 pad 15: unconnected-(J6-Pad15) -> /yellow_2
- J6 pad 16: unconnected-(J6-Pad16) -> GND
- J6 pad 17: unconnected-(J6-Pad17) -> /Green_2
- J6 pad 19: unconnected-(J6-Pad19) -> /Blue_2
- J6 pad 2: unconnected-(J6-Pad2) -> SDA
- J6 pad 20: unconnected-(J6-Pad20) -> GND
- J6 pad 21: unconnected-(J6-Pad21) -> /Black_2
- J6 pad 25: /yellow_2 -> GND
- J6 pad 27: /Green_2 -> /yellow_1
- J6 pad 29: /Blue_2 -> /Green_1
- J6 pad 30: unconnected-(J6-Pad30) -> STBY_1
- J6 pad 31: /Black_2 -> /Blue_1
- J6 pad 33: /yellow_1 -> /Black_1
- J6 pad 34: unconnected-(J6-Pad34) -> BIN1_1
- J6 pad 35: /Green_1 -> PWMA_1
- J6 pad 36: unconnected-(J6-Pad36) -> BIN2_1
- J6 pad 37: /Blue_1 -> AIN2_1
- J6 pad 39: /Black_1 -> AIN1_1
- J6 pad 40: unconnected-(J6-Pad40) -> PWMB_1
Routing:
- net STBY_1: track 0.00 -> 60.4 mm, vias 0 -> 1
- net +5V: track 117.3 -> 176.8 mm, vias 5 -> 6
- net BIN1_1: track 0.00 -> 55.8 mm, vias 0 -> 1
- net SDA: track 0.00 -> 54.1 mm
- net BIN2_1: track 0.00 -> 53.9 mm, vias 0 -> 1
- net PWMA_1: track 0.00 -> 51.0 mm
- net SCL: track 0.00 -> 51.0 mm
- net AIN2_1: track 0.00 -> 49.9 mm
- net PWMB_1: track 0.00 -> 49.5 mm
- net AIN1_1: track 0.00 -> 49.2 mm
- net GND: track 82.5 -> 120.7 mm, vias 100 -> 134
- net +12V: track 230.7 -> 206.7 mm
- net /Black_2: track 9.69 -> 19.5 mm
- net /Blue_2: track 9.43 -> 19.2 mm
- net /Green_2: track 8.90 -> 18.4 mm
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