File: extras/kicad/V2/Power/Power.kicad_pcb (KiCad board)
At the start: 2 copper layers, 181.3 x 110 mm, 77 parts, among them J1 Conn_01x02, J2 Screw_Terminal_01x06, J3 Screw_Terminal_01x06, J4 Screw_Terminal_01x06, J5 Screw_Terminal_01x06, J6 left, J7 right, U1 TB6612FNG, U2 TB6612FNG, U3 TPS5430DDAR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

Commit message: t
Parts:
- added C35: 22u, Capacitor_SMD:C_0805_2012Metric, B.Cu at (77.0, 105.4)
- added C36: 22u, Capacitor_SMD:C_0805_2012Metric, B.Cu at (74.9, 105.4)
- added C37: 22u, Capacitor_SMD:C_0805_2012Metric, B.Cu at (79.1, 105.4)
- added C38: 22u, Capacitor_SMD:C_0805_2012Metric, B.Cu at (74.9, 108.8)
- added C39: 22u, Capacitor_SMD:C_0805_2012Metric, B.Cu at (77.0, 108.8)
- added FID1: Fiducial, Fiducial:Fiducial_0.5mm_Mask1mm, F.Cu at (94.4, 136.9)
- added FID2: Fiducial, Symbol:WEEE-Logo_5.6x8mm_SilkScreen, F.Cu at (132.0, 119.4)
- added FID3: Fiducial, Symbol:OSHW-Logo2_14.6x12mm_SilkScreen, F.Cu at (159.0, 136.5)
- added FID4: Fiducial, Symbol:KiCad-Logo2_6mm_SilkScreen, F.Cu at (68.0, 135.4)
- added REF**: KiCad-Logo2_5mm_SilkScreen, Symbol:KiCad-Logo2_5mm_SilkScreen, B.Cu at (103.4, 86.3)
- added SW1: SW_SPST, Z_mycustom_footprint_lib:SPST Solder Plug Swith, F.Cu at (53.8, 101.2)
- added kibuzzard-63E93541: G***, kibuzzard-63E93541, B.Cu at (62.2, 124.7)
- added kibuzzard-63E93553: G***, kibuzzard-63E93553, B.Cu at (39.9, 110.9)
- moved C3 20.8 mm to (79.1, 108.8)
- moved J1 15.6 mm to (60.6, 113.2), turned to 180 degrees
- moved TP3 14.2 mm to (66.9, 115.4)
- moved TP4 14.2 mm to (70.1, 115.4)
- moved C1 14.2 mm to (68.5, 101.6)
- moved C2 14.2 mm to (72.2, 101.6)
- moved R12 14.2 mm to (68.5, 105.9)
- moved R13 14.2 mm to (68.5, 103.6)
- moved R2 14.2 mm to (68.5, 112.9)
- moved R7 14.2 mm to (68.5, 108.2)
- moved R9 14.2 mm to (68.5, 110.5)
- moved TP6 14.2 mm to (69.2, 91.8)
- moved TP5 14.2 mm to (67.1, 91.9)
- moved U5 14.2 mm to (69.8, 96.9)
Connections:
- C1 pad 2: Net-(J1-Pad2) -> Net-(C1-Pad2)
- J1 pad 2: Net-(J1-Pad2) -> /in
- R12 pad 1: Net-(J1-Pad2) -> Net-(C1-Pad2)
- R13 pad 1: Net-(J1-Pad2) -> Net-(C1-Pad2)
- R2 pad 1: Net-(J1-Pad2) -> Net-(C1-Pad2)
- R7 pad 1: Net-(J1-Pad2) -> Net-(C1-Pad2)
- R9 pad 1: Net-(J1-Pad2) -> Net-(C1-Pad2)
- TP3 pad 1: Net-(J1-Pad2) -> Net-(C1-Pad2)
- U5 pad 8: Net-(J1-Pad2) -> Net-(C1-Pad2)
Routing:
- net Net-(C1-Pad2): track 0.00 -> 26.6 mm
- net Net-(J1-Pad2): track 25.0 -> 0.00 mm
- net +5V: track 176.8 -> 162.4 mm
- net +12V: track 206.7 -> 193.5 mm
- net SDA: track 54.1 -> 49.2 mm
- net SCL: track 51.0 -> 46.5 mm
- net GND: track 120.7 -> 118.1 mm, vias 134 -> 154
- added copper zone on B.Cu, net +12V
- added copper zone on B.Cu, net /in
Other:
- board text added: "9-15V"
- board text added: "9-15v Battery LifePO4 recommended"
- board text added: "BLK"
- board text added: "BLU"
- board text added: "By Sniper1"
- board text added: "By Sniper2"
- board text added: "CERN-OHL-P"
- board text added: "DO NOT connect PI here!"
- board text added: "Eg Hacker TopFuel 3S LiPo 20C-ECO-X 2400mAh"
- board text added: "GND"
- board text added: "GRN"
- board text added: "Motor 1"
- board text added: "Motor 2"
- board text added: "Motor 3"
- board text added: "Motor 4"
- board text added: "RED"
- board text added: "Smartcar 2.0"
- board text added: "Smartcar 2.0 Motor board"
- board text added: "V_Batt"
- board text added: "WHT"
- board text added: "YLW"
- board text added: "github.com/immortal-sniper1"
- board text added: "rosmo-robot.github.io"

Commit message: g
Parts:
- added F1: Polyfuse, Fuse:Fuse_2920_7451Metric_Pad2.10x5.45mm_HandSolder, B.Cu at (46.1, 106.8)
- added J10: Conn_01x05, Connector_PinHeader_2.54mm:PinHeader_1x05_P2.54mm_Vertical, F.Cu at (39.9, -23.1)
- added J8: Conn_01x05, Connector_PinHeader_2.54mm:PinHeader_1x05_P2.54mm_Vertical, F.Cu at (47.6, 76.5)
- added J9: Conn_01x05, Connector_PinHeader_2.54mm:PinHeader_1x05_P2.54mm_Vertical, F.Cu at (43.0, 76.5)
- added R1: 10k, Resistor_SMD:R_0603_1608Metric, B.Cu at (114.0, 100.6)
- added R8: 10k, Resistor_SMD:R_0603_1608Metric, B.Cu at (114.0, 102.2)
- moved kibuzzard-63E93553 3.81 mm to (40.1, 114.7)
- moved REF** 3.00 mm to (106.4, 86.3)
Connections:
- J1 pad 2: /in -> Net-(J1-Pad2)
- J6 pad 3: GND -> INT
Routing:
- net +3V3: track 64.4 -> 114.4 mm, vias 2 -> 4
- net STBY_2: track 78.7 -> 103.5 mm, vias 0 -> 2
- net STBY_1: track 60.4 -> 82.6 mm, vias 1 -> 3
- net Net-(J1-Pad2): track 0.00 -> 10.5 mm
- net /in: track 0.00 -> 9.58 mm
- net +5V: track 162.4 -> 163.7 mm
- net GND: vias 154 -> 158
- removed copper zone on B.Cu, net /in

Commit message: t
Parts:
- removed J10: Conn_01x05, Connector_PinHeader_2.54mm:PinHeader_1x05_P2.54mm_Vertical
- moved J9 51.6 mm to (48.5, 127.8), turned to -135 degrees
- moved J8 8.71 mm to (48.4, 85.2), turned to -45 degrees
Connections:
- J7 pad 1: unconnected-(J7-Pad1) -> INT2
- J9 pad 2: INT -> INT2
Routing:
- net +3V3: track 114.4 -> 223.7 mm
- net SCL: track 46.5 -> 117.8 mm
- net SDA: track 49.2 -> 114.4 mm, vias 0 -> 1
- net INT: track 0.00 -> 62.9 mm
- net INT2: track 0.00 -> 57.8 mm

Commit message: t
Parts:
- added R10: 15k, Resistor_SMD:R_0603_1608Metric_Pad0.98x0.95mm_HandSolder, B.Cu at (96.2, 133.4)
- added R11: 150k, Resistor_SMD:R_0603_1608Metric_Pad0.98x0.95mm_HandSolder, B.Cu at (104.6, 65.5)
- R5: value 3k24 -> 2k2
- R6: value 5k9 -> 3k3
- moved TP1 1.33 mm to (93.8, 131.9)
Routing:
- net PWMB_2: track 71.0 -> 73.2 mm
- net BIN2_2: track 72.0 -> 73.7 mm
- net /3v3_FB: track 5.02 -> 6.64 mm
- net /5v_FB: track 5.18 -> 6.78 mm
- net BIN1_2: track 75.6 -> 77.0 mm
- net GND: track 118.1 -> 119.2 mm, vias 158 -> 2041
- net STBY_2: track 103.5 -> 104.5 mm
- net AIN1_2: track 76.6 -> 77.3 mm
- net Net-(TP1-Pad1): track 1.91 -> 2.45 mm
