File: extras/kicad/V2/Power/Power.kicad_sch (KiCad schematic)
At the start: 23 parts, among them J1 Conn_01x02, J2 Engine1, J3 Engine1, J4 Engine1, J5 Engine1, U1 TB6612FNG, U2 TB6612FNG

Commit message: g
Parts:
- added C13, C14, C? (x2): C_Small, symbol Device:C_Small
- added C15: 66u, symbol Device:C_Small
- added C16: 4n7, symbol Device:C_Small
- added C17, C?: 10n, symbol Device:C_Small
- added C18: 39p, symbol Device:C_Small
- added C?: 94u, symbol Device:C_Small
- added C? (x2): 100n, Capacitor_SMD:C_0603_1608Metric, symbol Device:C_Small
- added C?: 1n, symbol Device:C_Small
- added C?: 47p, symbol Device:C_Small
- added D1, D?: D_Small, symbol Device:D_Small
- added L1, L?: L_Small, symbol Device:L_Small
- added R2, R?: 1.2Meg, symbol Device:R_Small
- added R3, R?: 10k, symbol Device:R_Small
- added R4, R?: 120k, symbol Device:R_Small
- added R5: 1k91, symbol Device:R_Small
- added R6: 49.9, symbol Device:R_Small
- added R?: 3k24, symbol Device:R_Small
- added R?: 29.4, symbol Device:R_Small
- added U3, U?: TPS5430DDAR, Package_SO:SOIC-8-1EP_3.9x4.9mm_P1.27mm_EP2.29x3mm_ThermalVias, symbol My_custom_lib:TPS5430DDAR
- J3: value Engine1 -> Engine3
- J4: value Engine1 -> Engine2
- J5: value Engine1 -> Engine4
Connections:
- net +12V: now also C13.1, C14.1, C?.1, C?.1, R2.1, R?.1, U3.2 (VIN), U?.2 (VIN)
- net +3V3: now also C?.1, L?.2, R?.1
- net +5V: now also C15.1, L1.2, R3.1
- net GND: now also C13.2, C14.2, C15.2, C17.2, C18.2, C?.2, C?.2, C?.2, C?.2, C?.2, D1.2 (A), D?.2 (A), R4.2, R5.2, R6.2, R?.2, R?.2, R?.2, U3.7 (GND), U3.9 (Thermal), U?.7 (GND), U?.9 (Thermal)
- net PWMB_2: now reaches U2.15 (PWMB)
- net BIN2_2: now reaches U2.16 (BIN2)
- net BIN1_2: now reaches U2.17 (BIN1)
- net STBY_2: now reaches U2.19 (STBY)
- net AIN1_2: now reaches U2.21 (AIN1)
- net AIN2_2: now reaches U2.22 (AIN2)
- net PWMA_2: now reaches U2.23 (PWMA)
- net PWMB_1: now reaches U1.15 (PWMB)
- net BIN2_1: now reaches U1.16 (BIN2)
- net BIN1_1: now reaches U1.17 (BIN1)
- net STBY_1: now reaches U1.19 (STBY)
- net AIN1_1: now reaches U1.21 (AIN1)
- net AIN2_1: now reaches U1.22 (AIN2)
- net PWMA_1: now reaches U1.23 (PWMA)
- new net: R?.1, R?.2, U?.5 (VSENSE)
- new net: R?.1, R?.2, U?.3 (EN)
- new net: C16.1, R6.1
- new net: R3.2, R5.1, U3.5 (VSENSE)
- new net: R2.2, R4.1, U3.3 (EN)
- new net: C16.2, C18.1, U3.6 (COMP)
- new net: C?.2, D1.1 (K), L1.1, U3.8 (PH)
- new net: C?.1, U?.1 (BOOT)
- new net: C?.2, D?.1 (K), L?.1, U?.8 (PH)
- new net: C?.1, R?.1
- new net: C?.1, C?.2, U?.6 (COMP)
- new net: C?.1, U3.1 (BOOT)
- new net: C?.1, U?.4 (SS)
- new net: C17.1, U3.4 (SS)
Other:
- note added: "1.25V EN pin"
- moved on the sheet: C10, C11, C2, C4, C5, C6, C7, C8, C9, J2, J3, J4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

Commit message: g
Parts:
- removed C? (x2): C_Small, symbol Device:C_Small
- removed C?: 94u, symbol Device:C_Small
- removed D?: D_Small, symbol Device:D_Small
- removed J2: Engine1, symbol Connector_Generic:Conn_01x02
- removed J3: Engine3, symbol Connector_Generic:Conn_01x02
- removed J4: Engine2, symbol Connector_Generic:Conn_01x02
- removed J5: Engine4, symbol Connector_Generic:Conn_01x02
- removed R?: 1.2Meg, symbol Device:R_Small
- removed R?: 120k, symbol Device:R_Small
- added C19, C20, C23, C25, C26, C27, C28, C30: 22u, Capacitor_SMD:C_0805_2012Metric, symbol Device:C_Small
- added C21, C24, C29: 100n, Capacitor_SMD:C_0603_1608Metric, symbol Device:C_Small
- added D2: D, Diode_SMD:D_SMA, symbol Device:D_Small
- added H5, H6, H7, H8: Motor, Z_mycustom_footprint_lib:JGA25-370 DC motor, symbol Mechanical:MountingHole_Pad
- added J2, J3, J4, J5: Screw_Terminal_01x06, TerminalBlock_4Ucon:TerminalBlock_4Ucon_1x06_P3.50mm_Horizontal, symbol Connector:Screw_Terminal_01x06
- added J6, J7: Conn_02x20_Odd_Even, Connector_PinHeader_2.54mm:PinHeader_2x20_P2.54mm_Vertical, symbol Connector_Generic:Conn_02x20_Odd_Even
- added R12, R13, R7, R9: 0.1, Resistor_SMD:R_1206_3216Metric_Pad1.30x1.75mm_HandSolder, symbol Device:R_Small
- added R14, R15: 1Meg, Resistor_SMD:R_0603_1608Metric, symbol Device:R_Small
- added R16: 100k, Resistor_SMD:R_0603_1608Metric, symbol Device:R_Small
- C13: value C_Small -> 22u; footprint (none) -> Capacitor_SMD:C_0805_2012Metric; LCSC (none) -> C45783
- C14: value C_Small -> 100n; footprint (none) -> Capacitor_SMD:C_0603_1608Metric; LCSC (none) -> C14663
- C15: value 66u -> 22u; footprint (none) -> Capacitor_SMD:C_0805_2012Metric; LCSC (none) -> C45783
- D1: value D_Small -> D; footprint (none) -> Diode_SMD:D_SMA; LCSC (none) -> C22452
- J1: footprint (none) -> Connector_AMASS:AMASS_XT60-M_1x02_P7.20mm_Vertical
- R2: value 1.2Meg -> 0.1; footprint (none) -> Resistor_SMD:R_1206_3216Metric_Pad1.30x1.75mm_HandSolder; LCSC (none) -> C25334
- R3: footprint (none) -> Resistor_SMD:R_0603_1608Metric; LCSC (none) -> C25804
- R4: value 120k -> 100k; footprint (none) -> Resistor_SMD:R_0603_1608Metric; LCSC (none) -> C25803
- R8: renamed from R?; footprint (none) -> Resistor_SMD:R_0603_1608Metric; LCSC (none) -> C25804
- gave numbers to parts that had none: 9
Connections:
- net +12V: now also R2.2, C23.1, C24.1, R12.2, R13.2, R14.1, R15.1, R7.2, R9.2; no longer J1.2 (Pin_2), R2.1
- net +3V3: now also C25.1, C26.1, C27.1, C28.1, C29.1, C30.1
- net +5V: now also C19.1, C20.1, C21.1
- net GND: now also C19.2, C20.2, C21.2, C23.2, C24.2, C25.2, C26.2, C27.2, C28.2, C29.2, C30.2, D2.2 (A), H5.1, H6.1, H7.1, H8.1, R16.2
- net at U4.3 (EN): now also R15.2, R16.1
- net at R4.1, U3.3 (EN): now also R14.2; no longer R2.2
- net AO1_2: now reaches U2.1 (AO1), U2.2 (AO1)
- net AO1_2: now also J4.6 (Pin_6)
- net BO1_2: now reaches U2.11 (BO1), U2.12 (BO1)
- net BO1_2: now also J5.6 (Pin_6)
- net AO2_2: now reaches U2.5 (AO2), U2.6 (AO2)
- net AO2_2: now also J4.5 (Pin_5)
- net BO2_2: now reaches U2.7 (BO2), U2.8 (BO2)
- net BO2_2: now also J5.5 (Pin_5)
- net at C22.2, L2.1, U4.8 (PH): now also D2.1 (K)
- net AO1_1: now reaches U1.1 (AO1), U1.2 (AO1)
- net AO1_1: now also J2.6 (Pin_6)
- net BO1_1: now reaches U1.11 (BO1), U1.12 (BO1)
- net BO1_1: now also J3.6 (Pin_6)
- net AO2_1: now reaches U1.5 (AO2), U1.6 (AO2)
- net AO2_1: now also J2.5 (Pin_5)
- net BO2_1: now reaches U1.7 (BO2), U1.8 (BO2)
- net BO2_1: now also J3.5 (Pin_5)
- new net: J1.2 (Pin_2), R12.1, R13.1, R2.1, R7.1, R9.1
- new net Black_1: J2.1 (Pin_1)
- new net Black_2: J3.1 (Pin_1)
- new net Black_3: J4.1 (Pin_1)
- new net Black_4: J5.1 (Pin_1)
- new net Blue_1: J2.2 (Pin_2)
- new net Blue_2: J3.2 (Pin_2)
- new net Blue_3: J4.2 (Pin_2)
- new net Blue_4: J5.2 (Pin_2)
- new net Green_1: J2.3 (Pin_3)
- new net Green_2: J3.3 (Pin_3)
- new net Green_3: J4.3 (Pin_3)
- new net Green_4: J5.3 (Pin_3)
- new net yellow_1: J2.4 (Pin_4)
- new net yellow_2: J3.4 (Pin_4)
- new net yellow_3: J4.4 (Pin_4)
- new net yellow_4: J5.4 (Pin_4)
Other:
- moved on the sheet: C1, C10, C11, C12, C16, C17, C18, C22, C3, C31, C33, C4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

Commit message: f
Parts:
- C16, C17, C18, C31, C32, C33, R11, R6: footprint (none) -> Capacitor_SMD:C_0603_1608Metric_Pad1.08x0.95mm_HandSolder
- L1, L2: value L_Small -> 6u8; footprint (none) -> Z_mycustom_footprint_lib:Inductor SMD,11.6x10.1x4mm; LCSC (none) -> C3002684
- R10, R5: footprint (none) -> Resistor_SMD:R_0603_1608Metric_Pad0.98x0.95mm_HandSolder
Connections:
- net 3v3_FB: now reaches R10.1, R8.2, U4.5 (VSENSE)
- net 5v_FB: now reaches R3.2, R5.1, U3.5 (VSENSE)
- net EN1: now reaches R14.2, R4.1, U3.3 (EN)
- net EN2: now reaches R15.2, R16.1, U4.3 (EN)
- net ss2: now reaches C31.1, U4.4 (SS)
- net ss1: now reaches C17.1, U3.4 (SS)
Changed lines of the file:
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@@
+    (effects (font (size 1.27 1.27)) (justify left bottom))
+  )
+  (label "EN2" (at 76.2 226.06 0)
     (effects (font (size 1.27 1.27)) (justify left bottom))
   )
@@
     (effects (font (size 1.27 1.27)) (justify left bottom))
   )
+  (label "EN1" (at 74.93 167.64 0)
+    (effects (font (size 1.27 1.27)) (justify left bottom))
+  )
   (label "AO2_2" (at 217.17 83.82 0)
     (effects (font (size 1.27 1.27)) (justify left bottom))
@@
     (effects (font (size 1.27 1.27)) (justify left bottom))
   )
+  (label "ss2" (at 76.2 229.87 0)
+    (effects (font (size 1.27 1.27)) (justify left bottom))
+  )
   (label "Black_4" (at 370.84 74.93 0)
     (effects (font (size 1.27 1.27)) (justify left bottom))
@@
     (effects (font (size 1.27 1.27)) (justify left bottom))
   )
+  (label "5v_FB" (at 124.46 175.26 0)
+    (effects (font (size 1.27 1.27)) (justify left bottom))
+  )
   (label "Green_1" (at 264.16 69.85 0)
     (effects (font (size 1.27 1.27)) (justify left bottom))
@@
     (effects (font (size 1.27 1.27)) (justify left bottom))
   )
+  (label "3v3_FB" (at 121.92 233.68 0)
+    (effects (font (size 1.27 1.27)) (justify left bottom))
+  )
   (label "BO2_2" (at 370.84 64.77 0)
     (effects (font (size 1.27 1.27)) (justify left bottom))
@@
   )
   (label "AO1_2" (at 217.17 78.74 0)
+    (effects (font (size 1.27 1.27)) (justify left bottom))
+  )
+  (label "ss1" (at 78.74 171.45 0)
     (effects (font (size 1.27 1.27)) (justify left bottom))
   )
@@
       (effects (font (size 1.27 1.27)) (justify left))
     )
-    (property "Footprint" "" (id 2) (at 82.55 190.5 0)
+    (property "Footprint" "Capacitor_SMD:C_0603_1608Metric_Pad1.08x0.95mm_HandSolder" (id 2) (at 82.55 190.5 0)
       (effects (font (size 1.27 1.27)) hide)
     )
@@
       (effects (font (size 1.27 1.27)) (justify left))
     )
-    (property "Footprint" "" (id 2) (at 133.35 179.07 0)
+    (property "Footprint" "Resistor_SMD:R_0603_1608Metric_Pad0.98x0.95mm_HandSolder" (id 2) (at 133.35 179.07 0)
       (effects (font (size 1.27 1.27)) hide)
     )
@@
       (effects (font (size 1.27 1.27)) (justify left))
     )
-    (property "Footprint" "" (id 2) (at 82.55 184.15 0)
+    (property "Footprint" "Capacitor_SMD:C_0603_1608Metric_Pad1.08x0.95mm_HandSolder" (id 2) (at 82.55 184.15 0)
       (effects (font (size 1.27 1.27)) hide)
     )
@@
     (in_bom yes) (on_board yes)
     (property "Reference" "L1" (id 0) (at 125.73 165.735 90))
-    (property "Value" "L_Small" (id 1) (at 125.73 168.275 90))
-    (property "Footprint" "" (id 2) (at 125.73 163.83 0)
-      (effects (font (size 1.27 1.27)) hide)
-    )
-    (property "Datasheet" "~" (id 3) (at 125.73 163.83 0)
+    (property "Value" "6u8" (id 1) (at 125.73 168.275 90))
+    (property "Footprint" "Z_mycustom_footprint_lib:Inductor SMD,11.6x10.1x4mm" (id 2) (at 125.73 163.83 0)
+      (effects (font (size 1.27 1.27)) hide)
+    )
+    (property "Datasheet" "https://jlcpcb.com/partdetail/Cenker-CKST1004_6_8uH_MNCK/C3002684" (id 3) (at 125.73 163.83 0)
+      (effects (font (size 1.27 1.27)) hide)
+    )
+    (property "LCSC" "C3002684" (id 4) (at 125.73 163.83 90)
       (effects (font (size 1.27 1.27)) hide)
     )
@@
       (effects (font (size 1.27 1.27)) (justify left))
     )
-    (property "Footprint" "" (id 2) (at 78.74 184.15 0)
+    (property "Footprint" "Capacitor_SMD:C_0603_1608Metric_Pad1.08x0.95mm_HandSolder" (id 2) (at 78.74 184.15 0)
       (effects (font (size 1.27 1.27)) hide)
     )
@@
       (effects (font (size 1.27 1.27)) (justify left))
     )
-    (property "Footprint" "" (id 2) (at 82.55 242.57 0)
+    (property "Footprint" "Capacitor_SMD:C_0603_1608Metric_Pad1.08x0.95mm_HandSolder" (id 2) (at 82.55 242.57 0)
       (effects (font (size 1.27 1.27)) hide)
     )
@@
       (effects (font (size 1.27 1.27)) (justify left))
     )
-    (property "Footprint" "" (id 2) (at 132.08 238.76 0)
+    (property "Footprint" "Resistor_SMD:R_0603_1608Metric_Pad0.98x0.95mm_HandSolder" (id 2) (at 132.08 238.76 0)
       (effects (font (size 1.27 1.27)) hide)
     )
@@
       (effects (font (size 1.27 1.27)) (justify left))
     )
-    (property "Footprint" "" (id 2) (at 68.58 242.57 0)
+    (property "Footprint" "Capacitor_SMD:C_0603_1608Metric_Pad1.08x0.95mm_HandSolder" (id 2) (at 68.58 242.57 0)
       (effects (font (size 1.27 1.27)) hide)
     )
@@
       (effects (font (size 1.27 1.27)) (justify left))
     )
-    (property "Footprint" "" (id 2) (at 77.47 242.57 0)
+    (property "Footprint" "Capacitor_SMD:C_0603_1608Metric_Pad1.08x0.95mm_HandSolder" (id 2) (at 77.47 242.57 0)
       (effects (font (size 1.27 1.27)) hide)
     )
@@
       (effects (font (size 1.27 1.27)) (justify left))
     )
-    (property "Footprint" "" (id 2) (at 82.55 250.19 0)
+    (property "Footprint" "Capacitor_SMD:C_0603_1608Metric_Pad1.08x0.95mm_HandSolder" (id 2) (at 82.55 250.19 0)
       (effects (font (size 1.27 1.27)) hide)
     )
@@
       (effects (font (size 1.27 1.27)) (justify left))
     )
-    (property "Footprint" "" (id 2) (at 68.58 184.15 0)
+    (property "Footprint" "Capacitor_SMD:C_0603_1608Metric_Pad1.08x0.95mm_HandSolder" (id 2) (at 68.58 184.15 0)
       (effects (font (size 1.27 1.27)) hide)
     )
@@
     )
     (property "LCSC" "C25334" (id 4) (at 40.64 31.75 90)
-      (effects (font (size 1.27 1.27)) hide)
-    )
-    (pin "1")
-    (pin "2")
-  )
-  (symbol (lib_id "Device:L_Small") (at 125.73 222.25 90) (unit 1)
-    (in_bom yes) (on_board yes)
-    (property "Reference" "L2" (id 0) (at 125.73 224.155 90))
-    (property "Value" "L_Small" (id 1) (at 125.73 226.695 90))
-    (property "Footprint" "" (id 2) (at 125.73 222.25 0)
-      (effects (font (size 1.27 1.27)) hide)
-    )
-    (property "Datasheet" "~" (id 3) (at 125.73 222.25 0)
       (effects (font (size 1.27 1.27)) hide)
     )
@@
     (pin "1")
   )
+  (symbol (lib_id "Device:L_Small") (at 125.73 222.25 90) (unit 1)
+    (in_bom yes) (on_board yes)
+    (property "Reference" "L2" (id 0) (at 125.73 224.155 90))
+    (property "Value" "6u8" (id 1) (at 125.73 226.695 90))
+    (property "Footprint" "Z_mycustom_footprint_lib:Inductor SMD,11.6x10.1x4mm" (id 2) (at 125.73 222.25 0)
+      (effects (font (size 1.27 1.27)) hide)
+    )
+    (property "Datasheet" "https://jlcpcb.com/partdetail/Cenker-CKST1004_6_8uH_MNCK/C3002684" (id 3) (at 125.73 222.25 0)
+      (effects (font (size 1.27 1.27)) hide)
+    )
+    (property "LCSC" "C3002684" (id 4) (at 125.73 222.25 90)
+      (effects (font (size 1.27 1.27)) hide)
+    )
+    (pin "1")
+    (pin "2")
+  )
   (symbol (lib_id "Connector_Generic:Conn_01x02") (at 19.05 41.91 180) (unit 1)
     (in_bom yes) (on_board yes) (fields_autoplaced)
@@
     )
     (path "/1f4dc53b-1e0a-4367-9539-e28149c7c0a5"
-      (reference "C16") (unit 1) (value "4n7") (footprint "")
+      (reference "C16") (unit 1) (value "4n7") (footprint "Capacitor_SMD:C_0603_1608Metric_Pad1.08x0.95mm_HandSolder")
     )
     (path "/c45fe646-0896-45b5-819f-e5e557d951a3"
-      (reference "C17") (unit 1) (value "10n") (footprint "")
+      (reference "C17") (unit 1) (value "10n") (footprint "Capacitor_SMD:C_0603_1608Metric_Pad1.08x0.95mm_HandSolder")
     )
     (path "/217c59c9-7ddd-4a55-a18d-81abc3edec31"
-      (reference "C18") (unit 1) (value "39p") (footprint "")
+      (reference "C18") (unit 1) (value "39p") (footprint "Capacitor_SMD:C_0603_1608Metric_Pad1.08x0.95mm_HandSolder")
     )
     (path "/0382afdf-0016-4a76-87d2-368a7c541fe8"
@@
     )
     (path "/738a367b-ddc2-41fa-ac7f-36ddf30931ef"
-      (reference "C31") (unit 1) (value "10n") (footprint "")
+      (reference "C31") (unit 1) (value "10n") (footprint "Capacitor_SMD:C_0603_1608Metric_Pad1.08x0.95mm_HandSolder")
     )
     (path "/a7872e69-b3ab-49e8-9be6-0841937b4ef8"
-      (reference "C32") (unit 1) (value "47p") (footprint "")
+      (reference "C32") (unit 1) (value "47p") (footprint "Capacitor_SMD:C_0603_1608Metric_Pad1.08x0.95mm_HandSolder")
     )
     (path "/45cb49d9-0608-4ed8-a6f2-4e7d2734b351"
-      (reference "C33") (unit 1) (value "1n") (footprint "")
+      (reference "C33") (unit 1) (value "1n") (footprint "Capacitor_SMD:C_0603_1608Metric_Pad1.08x0.95mm_HandSolder")
     )
     (path "/3ff02452-e10e-4ce1-b274-f1acc6de8b8c"
@@
     )
     (path "/20386b90-ea74-450b-9374-e1b5bc66a2a4"
-      (reference "L1") (unit 1) (value "L_Small") (footprint "")
-    )
-    (path "/d1524a72-f599-4186-8986-cfeae0c1753a"
-      (reference "L2") (unit 1) (value "L_Small") (footprint "")
+      (reference "L1") (unit 1) (value "6u8") (footprint "Z_mycustom_footprint_lib:Inductor SMD,11.6x10.1x4mm")
+    )
+    (path "/f683613a-63bf-4150-8477-1cbc8e4fc079"
+      (reference "L2") (unit 1) (value "6u8") (footprint "Z_mycustom_footprint_lib:Inductor SMD,11.6x10.1x4mm")
     )
     (path "/0b8ad130-b85a-4d2e-9d43-2240caedc79b"
@@
     )
     (path "/0fdda146-07d6-47a9-89bf-c945bd5bec51"
-      (reference "R5") (unit 1) (value "1k91") (footprint "")
+      (reference "R5") (unit 1) (value "1k91") (footprint "Resistor_SMD:R_0603_1608Metric_Pad0.98x0.95mm_HandSolder")
     )
     (path "/05317954-b415-4b64-ada7-cfbaa23dbe4d"
-      (reference "R6") (unit 1) (value "49.9") (footprint "")
+      (reference "R6") (unit 1) (value "49.9") (footprint "Capacitor_SMD:C_0603_1608Metric_Pad1.08x0.95mm_HandSolder")
     )
     (path "/ceb33d94-18cc-4d50-ac9e-eebe4a271d7f"
@@
     )
     (path "/719facbd-9f8d-4a24-85e8-4721909281b0"
-      (reference "R10") (unit 1) (value "3k24") (footprint "")
+      (reference "R10") (unit 1) (value "3k24") (footprint "Resistor_SMD:R_0603_1608Metric_Pad0.98x0.95mm_HandSolder")
     )
     (path "/bea2d2e9-ff61-4860-97ec-c2b169e59d9c"
-      (reference "R11") (unit 1) (value "29.4") (footprint "")
+      (reference "R11") (unit 1) (value "29.4") (footprint "Capacitor_SMD:C_0603_1608Metric_Pad1.08x0.95mm_HandSolder")
     )
     (path "/d8549c68-6479-46b2-9db2-cbe6d76aaedd"

Commit message: t
Parts:
- removed C16: 4n7, Capacitor_SMD:C_0603_1608Metric_Pad1.08x0.95mm_HandSolder, symbol Device:C_Small
- removed C17, C31: 10n, Capacitor_SMD:C_0603_1608Metric_Pad1.08x0.95mm_HandSolder, symbol Device:C_Small
- removed C18: 39p, Capacitor_SMD:C_0603_1608Metric_Pad1.08x0.95mm_HandSolder, symbol Device:C_Small
- removed C22, C24, C29: 100n, Capacitor_SMD:C_0603_1608Metric, symbol Device:C_Small
- removed C23, C25, C26, C27, C28, C30: 22u, Capacitor_SMD:C_0805_2012Metric, symbol Device:C_Small
- removed C32: 47p, Capacitor_SMD:C_0603_1608Metric_Pad1.08x0.95mm_HandSolder, symbol Device:C_Small
- removed C33: 1n, Capacitor_SMD:C_0603_1608Metric_Pad1.08x0.95mm_HandSolder, symbol Device:C_Small
- removed D2: D, Diode_SMD:D_SMA, symbol Device:D_Small
- removed L2: 6u8, Z_mycustom_footprint_lib:Inductor SMD,11.6x10.1x4mm, symbol Device:L_Small
- removed R10: 3k24, Resistor_SMD:R_0603_1608Metric_Pad0.98x0.95mm_HandSolder, symbol Device:R_Small
- removed R11: 29.4, Capacitor_SMD:C_0603_1608Metric_Pad1.08x0.95mm_HandSolder, symbol Device:R_Small
- removed R14, R15: 1Meg, Resistor_SMD:R_0603_1608Metric, symbol Device:R_Small
- removed R16, R4: 100k, Resistor_SMD:R_0603_1608Metric, symbol Device:R_Small
- removed R6: 49.9, Capacitor_SMD:C_0603_1608Metric_Pad1.08x0.95mm_HandSolder, symbol Device:R_Small
- removed R8: 10k, Resistor_SMD:R_0603_1608Metric, symbol Device:R_Small
- removed U4: TPS5430DDAR, Package_SO:SOIC-8-1EP_3.9x4.9mm_P1.27mm_EP2.29x3mm_ThermalVias, symbol My_custom_lib:TPS5430DDAR
Connections:
- net ss1 is gone; now on net 5v_FB: U3.4 (VSENSE)
- net +12V: now also U3.7 (Vin); no longer U3.2 (VIN)
- net 5v_FB: no longer U3.5 (VSENSE)
- net GND: now also U3.6 (GND); no longer U3.7 (GND)
- net at D1.1 (K), L1.1, U3.8 (PH): now also C12.1; no longer C12.2
- net at U3.1 (BOOT): now also C12.2; no longer C12.1
- net EN1: no longer names the net of U3.3 (NC)
Other:
- note added: "under 0.5V to disable"
- note removed: "1.25V EN pin"
- moved on the sheet: C12, C13, C14, D1

Commit message: n
Parts:
- added C16, C26: 1n5, Capacitor_SMD:C_0603_1608Metric_Pad1.08x0.95mm_HandSolder, symbol Device:C_Small
- added C17, C18, C22, C24, C27, C28, C29, C30, C31, C32, C33: 47u, Capacitor_SMD:C_1206_3216Metric, symbol Device:C_Small
- added C23, C25, C34: 100n, Capacitor_SMD:C_0603_1608Metric, symbol Device:C_Small
- added D2: D, Diode_SMD:D_SMA, symbol Device:D_Small
- added L2: 15u, Z_mycustom_footprint_lib:Inductor SMD,11.6x10.1x4mm, symbol Device:L_Small
- added R4: 10k, Resistor_SMD:R_0603_1608Metric, symbol Device:R_Small
- added R6: 5k9, Resistor_SMD:R_0603_1608Metric_Pad0.98x0.95mm_HandSolder, symbol Device:R_Small
- added TP1, TP2: TestPoint, TestPoint:TestPoint_Pad_D1.0mm, symbol Connector:TestPoint
- added U4: TPS5430DDAR, Package_SO:SOIC-8-1EP_3.9x4.9mm_P1.27mm_EP2.29x3mm_ThermalVias, symbol My_custom_lib:TPS5430DDAR
- C1: value C_Small -> 1n5; footprint (none) -> Capacitor_SMD:C_0603_1608Metric_Pad1.08x0.95mm_HandSolder
- C13, C15, C19, C20: value 22u -> 47u; footprint Capacitor_SMD:C_0805_2012Metric -> Capacitor_SMD:C_1206_3216Metric; LCSC C45783 -> C96123
- L1: value 6u8 -> 15u; LCSC C3002684 -> C3002687
- R5: value 1k91 -> 3k24
Connections:
- net +12V: now also C24.1, C25.1, U4.7 (Vin)
- net +3V3: now also C26.1, C27.1, C28.1, C29.1, C30.1, C31.1, C32.1, C33.1, C34.1, L2.2, R4.1
- net +5V: now also C16.1, C17.1, C18.1, C22.1
- net 5v_FB: now also C16.2
- net GND: now also C17.2, C18.2, C22.2, C24.2, C25.2, C27.2, C28.2, C29.2, C30.2, C31.2, C32.2, C33.2, C34.2, D2.2 (A), R6.2, U4.6 (GND), U4.9 (Thermal)
- net at U3.5 (ENA): now also TP1.1
- new net: C23.1, D2.1 (K), L2.1, U4.8 (PH)
- new net: TP2.1, U4.5 (ENA)
- new net: C23.2, U4.1 (BOOT)
- new net 3v3_FB: C26.2, R4.2, R6.1, U4.4 (VSENSE)
Other:
- moved on the sheet: C15, C21

Commit message: g
Parts:
- added H10, H11, H12, H9: Bumper, MountingHole:MountingHole_4.5mm, symbol Mechanical:MountingHole
Connections:
- net +3V3: now also J6.5 (Pin_5), J6.6 (Pin_6), J6.7 (Pin_7), J6.8 (Pin_8)
- net +5V: now also J7.13 (Pin_13), J7.14 (Pin_14), J7.15 (Pin_15), J7.16 (Pin_16)
- net AO1_1: now also J3.6 (Pin_6); no longer J2.6 (Pin_6)
- net AO1_2: now also J4.5 (Pin_5); no longer J4.6 (Pin_6)
- net AO2_1: now also J3.5 (Pin_5); no longer J2.5 (Pin_5)
- net AO2_2: now also J4.6 (Pin_6); no longer J4.5 (Pin_5)
- net BO1_1: now also J2.5 (Pin_5); no longer J3.6 (Pin_6)
- net BO2_1: now also J2.6 (Pin_6); no longer J3.5 (Pin_5)
- net Black_1: now also J6.39 (Pin_39)
- net Black_2: now also J6.31 (Pin_31)
- net Black_3: now also J7.40 (Pin_40)
- net Black_4: now also J7.32 (Pin_32)
- net Blue_1: now also J6.37 (Pin_37)
- net Blue_2: now also J6.29 (Pin_29)
- net Blue_3: now also J7.38 (Pin_38)
- net Blue_4: now also J7.30 (Pin_30)
- net GND: now also J6.10 (Pin_10), J6.26 (Pin_26), J6.3 (Pin_3), J6.32 (Pin_32), J6.38 (Pin_38), J6.4 (Pin_4), J6.9 (Pin_9), J7.11 (Pin_11), J7.12 (Pin_12), J7.17 (Pin_17), J7.18 (Pin_18), J7.25 (Pin_25), J7.31 (Pin_31), J7.37 (Pin_37)
- net Green_1: now also J6.35 (Pin_35)
- net Green_2: now also J6.27 (Pin_27)
- net Green_3: now also J7.36 (Pin_36)
- net Green_4: now also J7.28 (Pin_28)
- net yellow_1: now also J6.33 (Pin_33)
- net yellow_2: now also J6.25 (Pin_25)
- net yellow_3: now also J7.34 (Pin_34)
- net yellow_4: now also J7.26 (Pin_26)
Other:
- moved on the sheet: J6, J7
