File: extras/kicad/V2/Power/Power.kicad_sch (KiCad schematic)
At the start: 77 parts, among them J1 Conn_01x02, J2 Screw_Terminal_01x06, J3 Screw_Terminal_01x06, J4 Screw_Terminal_01x06, J5 Screw_Terminal_01x06, J6 left, J7 right, U1 TB6612FNG, U2 TB6612FNG, U3 TPS5430DDAR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

Commit message: t
Parts:
- added C35, C36, C37, C38, C39: 22u, Capacitor_SMD:C_0805_2012Metric, symbol Device:C_Small
- added FID1: Fiducial, Fiducial:Fiducial_0.5mm_Mask1mm, symbol Mechanical:Fiducial
- added FID2: Fiducial, Symbol:WEEE-Logo_5.6x8mm_SilkScreen, symbol Mechanical:Fiducial
- added FID3: Fiducial, Symbol:OSHW-Logo2_14.6x12mm_SilkScreen, symbol Mechanical:Fiducial
- added FID4: Fiducial, Symbol:KiCad-Logo2_6mm_SilkScreen, symbol Mechanical:Fiducial
- added SW1: SW_SPST, Z_mycustom_footprint_lib:SPST Solder Plug Swith, symbol Switch:SW_SPST
Connections:
- net +12V: now also C35.1, C36.1, C37.1, C38.1, C39.1
- net GND: now also C35.2, C36.2, C37.2, C38.2, C39.2
- net at C1.2, R12.1, R13.1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: now also SW1.2 (B); no longer J1.2 (Pin_2)
- new net in: J1.2 (Pin_2), SW1.1 (A)
Other:
- moved on the sheet: C1, C10, C11, C2, C3, C4, C5, C6, C7, C8, C9, J1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

Commit message: g
Parts:
- added F1: Polyfuse, Fuse:Fuse_2920_7451Metric_Pad2.10x5.45mm_HandSolder, symbol Device:Polyfuse
- added J10, J8, J9: Conn_01x05, Connector_PinHeader_2.54mm:PinHeader_1x05_P2.54mm_Vertical, symbol Connector_Generic:Conn_01x05
- added R1, R8: 10k, Resistor_SMD:R_0603_1608Metric, symbol Device:R_Small
Connections:
- net +3V3: now also J10.5 (Pin_5), J8.5 (Pin_5), J9.5 (Pin_5), R1.1, R8.1
- net GND: now also J10.1 (Pin_1), J8.1 (Pin_1), J9.1 (Pin_1); no longer J6.3 (Pin_3)
- net SCL: now also J10.3 (Pin_3), J8.3 (Pin_3), J9.3 (Pin_3)
- net SDA: now also J10.4 (Pin_4), J8.4 (Pin_4), J9.4 (Pin_4)
- net STBY_1: now also R1.2
- net STBY_2: now also R8.2
- net in: now also F1.2; no longer J1.2 (Pin_2)
- new net: F1.1, J1.2 (Pin_2)
- new net INT: J10.2 (Pin_2), J6.3 (Pin_3), J8.2 (Pin_2), J9.2 (Pin_2)
Other:
- moved on the sheet: C1, C2, C3, C35, C36, C37, C38, C39, J1, R12, R13, R2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

Commit message: t
Parts:
- removed J10: Conn_01x05, Connector_PinHeader_2.54mm:PinHeader_1x05_P2.54mm_Vertical, symbol Connector_Generic:Conn_01x05
Connections:
- net INT: no longer J9.2 (Pin_2)
- net INT2: now reaches J7.1 (Pin_1)
- net INT2: now also J9.2 (Pin_2)
Other:
- note added: "Battery"
- note added: "Holes+ Markers"
- note added: "IO"
- note added: "Motor Drivvers"
- note added: "Motor IO"
- note added: "Power"
- note added: "PullUPS"
- moved on the sheet: C1, C10, C11, C12, C13, C14, C15, C16, C17, C18, C19, C2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

Commit message: t
Parts:
- added R10: 15k, Resistor_SMD:R_0603_1608Metric_Pad0.98x0.95mm_HandSolder, symbol Device:R_Small
- added R11: 150k, Resistor_SMD:R_0603_1608Metric_Pad0.98x0.95mm_HandSolder, symbol Device:R_Small
- C16, C26: LCSC (none) -> C1595
- R5: value 3k24 -> 2k2; LCSC (none) -> C4190
- R6: value 5k9 -> 3k3; LCSC (none) -> C22978
Connections:
- net 3v3_FB: now also R11.1
- net 5v_FB: now also R10.1
- net GND: now also R10.2, R11.2

Commit message: i
Parts:
- removed J1: Conn_01x02, Connector_AMASS:AMASS_XT60-M_1x02_P7.20mm_Vertical, symbol Connector_Generic:Conn_01x02
- removed SW1: SW_SPST, Z_mycustom_footprint_lib:SPST Solder Plug Swith, symbol Switch:SW_SPST
- added J1: XT60PW-M, footprint:CONN-TH_XT60PW-M, symbol My_Schematic_lib:XT60PW-M
- added SW1: SS01-BBIWA-RA20-R, footprint:SW-TH_SS01-BBIWA-RA20-R, symbol My_Schematic_lib:SS01-BBIWA-RA20-R
Connections:
- net GND: now also J1.1 (-)
- net in: now also SW1.1
- net at C1.2, R12.1, R13.1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: now also SW1.2
- net at F1.1: now also J1.2 (+)
- no-connect marks 0 -> 2
Changed lines of the file:
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@@
   (junction (at 309.88 39.37) (diameter 0) (color 0 0 0 0)
   )
+  (no_connect (at 22.86 50.8))
+  (no_connect (at 22.86 38.1))
   (wire (pts (xy 128.27 30.48) (xy 128.27 33.02))
     (stroke (width 0) (type default) (color 0 0 0 0))
@@
     (stroke (width 0) (type default) (color 0 0 0 0))
   )
+  (wire (pts (xy 66.04 43.18) (xy 72.39 43.18))
+    (stroke (width 0) (type default) (color 0 0 0 0))
+  )
   (wire (pts (xy 238.76 35.56) (xy 241.3 35.56))
     (stroke (width 0) (type default) (color 0 0 0 0))
@@
     (stroke (width 0) (type default) (color 0 0 0 0))
   )
-  (wire (pts (xy 45.72 43.18) (xy 54.61 43.18))
+  (wire (pts (xy 45.72 43.18) (xy 50.8 43.18))
     (stroke (width 0) (type default) (color 0 0 0 0))
   )
@@
     (stroke (width 0) (type default) (color 0 0 0 0))
   )
-  (wire (pts (xy 64.77 43.18) (xy 72.39 43.18))
-    (stroke (width 0) (type default) (color 0 0 0 0))
-  )
   (wire (pts (xy 69.85 158.75) (xy 64.77 158.75))
     (stroke (width 0) (type default) (color 0 0 0 0))
@@
     (pin "1")
   )
-  (symbol (lib_id "Switch:SW_SPST") (at 59.69 43.18 0) (unit 1)
-    (in_bom yes) (on_board yes) (fields_autoplaced)
-    (property "Reference" "SW1" (id 0) (at 59.69 36.83 0))
-    (property "Value" "SW_SPST" (id 1) (at 59.69 39.37 0))
-    (property "Footprint" "Z_mycustom_footprint_lib:SPST Solder Plug Swith" (id 2) (at 59.69 43.18 0)
-      (effects (font (size 1.27 1.27)) hide)
-    )
-    (property "Datasheet" "https://jlcpcb.com/parts/componentSearch?searchTxt=C309065" (id 3) (at 59.69 43.18 0)
-      (effects (font (size 1.27 1.27)) hide)
-    )
-    (property "LCSC" "C309065" (id 4) (at 59.69 43.18 0)
-      (effects (font (size 1.27 1.27)) hide)
-    )
-    (pin "1")
-    (pin "2")
-  )
   (symbol (lib_id "power:GND") (at 55.88 252.73 90) (unit 1)
     (in_bom yes) (on_board yes) (fields_autoplaced)
@@
     (pin "9")
   )
+  (symbol (lib_id "My_Schematic_lib:XT60PW-M") (at 26.67 41.91 180) (unit 1)
+    (in_bom yes) (on_board yes)
+    (property "Reference" "J1" (id 0) (at 29.845 33.02 0)
+      (effects (font (size 1.27 1.27)) (justify left))
+    )
+    (property "Value" "XT60PW-M" (id 1) (at 29.845 35.56 0)
+      (effects (font (size 1.27 1.27)) (justify left))
+    )
+    (property "Footprint" "footprint:CONN-TH_XT60PW-M" (id 2) (at 26.67 31.75 0)
+      (effects (font (size 1.27 1.27) italic) hide)
+    )
+    (property "Datasheet" "https://atta.szlcsc.com/upload/public/pdf/source/20180125/C98732_15168617837851301983.pdf" (id 3) (at 28.956 42.037 0)
+      (effects (font (size 1.27 1.27)) (justify left) hide)
+    )
+    (property "LCSC" "C98732" (id 4) (at 26.67 41.91 0)
+      (effects (font (size 1.27 1.27)) hide)
+    )
+    (pin "1")
+    (pin "2")
+    (pin "3")
+    (pin "4")
+  )
   (symbol (lib_id "power:GND") (at 334.01 91.44 0) (unit 1)
     (in_bom yes) (on_board yes) (fields_autoplaced)
@@
     (pin "1")
   )
+  (symbol (lib_id "My_Schematic_lib:SS01-BBIWA-RA20-R") (at 58.42 43.18 0) (unit 1)
+    (in_bom yes) (on_board yes) (fields_autoplaced)
+    (property "Reference" "SW1" (id 0) (at 58.42 35.56 0))
+    (property "Value" "SS01-BBIWA-RA20-R" (id 1) (at 58.42 38.1 0))
+    (property "Footprint" "footprint:SW-TH_SS01-BBIWA-RA20-R" (id 2) (at 58.42 53.34 0)
+      (effects (font (size 1.27 1.27) italic) hide)
+    )
+    (property "Datasheet" "https://item.szlcsc.com/292826.html" (id 3) (at 56.134 43.053 0)
+      (effects (font (size 1.27 1.27)) (justify left) hide)
+    )
+    (property "LCSC" "C309065" (id 4) (at 58.42 43.18 0)
+      (effects (font (size 1.27 1.27)) hide)
+    )
+    (pin "1")
+    (pin "2")
+  )
   (symbol (lib_id "power:+12V") (at 162.56 36.83 0) (unit 1)
     (in_bom yes) (on_board yes) (fields_autoplaced)
@@
     (pin "1")
   )
-  (symbol (lib_id "Connector_Generic:Conn_01x02") (at 26.67 45.72 180) (unit 1)
-    (in_bom yes) (on_board yes) (fields_autoplaced)
-    (property "Reference" "J1" (id 0) (at 26.67 36.83 0))
-    (property "Value" "Conn_01x02" (id 1) (at 26.67 39.37 0))
-    (property "Footprint" "Connector_AMASS:AMASS_XT60-M_1x02_P7.20mm_Vertical" (id 2) (at 26.67 45.72 0)
-      (effects (font (size 1.27 1.27)) hide)
-    )
-    (property "Datasheet" "~" (id 3) (at 26.67 45.72 0)
-      (effects (font (size 1.27 1.27)) hide)
-    )
-    (pin "1")
-    (pin "2")
-  )
   (symbol (lib_id "power:GND") (at 173.99 48.26 0) (unit 1)
     (in_bom yes) (on_board yes) (fields_autoplaced)
@@
       (reference "H12") (unit 1) (value "Bumper") (footprint "MountingHole:MountingHole_4.5mm")
     )
-    (path "/f7f52bc5-b406-4e8f-9473-907f39b2a6d0"
-      (reference "J1") (unit 1) (value "Conn_01x02") (footprint "Connector_AMASS:AMASS_XT60-M_1x02_P7.20mm_Vertical")
+    (path "/6114e62a-b0e5-4531-98d2-70e0db2ebbfb"
+      (reference "J1") (unit 1) (value "XT60PW-M") (footprint "footprint:CONN-TH_XT60PW-M")
     )
     (path "/cd8695d2-300e-4c23-b3ea-77e46f75b7b6"
@@
       (reference "R13") (unit 1) (value "0.1") (footprint "Resistor_SMD:R_1206_3216Metric_Pad1.30x1.75mm_HandSolder")
     )
-    (path "/33405962-7f3e-45ad-9d44-6a37428867ea"
-      (reference "SW1") (unit 1) (value "SW_SPST") (footprint "Z_mycustom_footprint_lib:SPST Solder Plug Swith")
+    (path "/f06685c4-d568-4470-ba5d-78a169218f3d"
+      (reference "SW1") (unit 1) (value "SS01-BBIWA-RA20-R") (footprint "footprint:SW-TH_SS01-BBIWA-RA20-R")
     )
     (path "/b30be24d-7e8e-4ff4-a3ac-03919a574b45"
