File: extras/kicad/V2/Control/Control.kicad_sch (KiCad schematic)
At the start: 50 parts, among them J1 Ultrasonic Ranging, J2 Conn_01x05, J3 Output, J4 Input, J6 left, J7 right, P8 BeagleBone_Black_Header, P9 BeagleBone_Black_Header, U1 SparkFun-micromod, U3 LIS3DHTR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

Commit message: Update Control.kicad_sch
Connections:
- net INT is gone; now on net INT_1: J2.2 (Pin_2)
- net +3V3: now also J?.1 (3V3)
- net D2+: now also U1.3 (USB_D+)
- net D2-: now also U1.5 (USB_D-)
- net GND: now also J?.2 (GND)
- net Green_1: now also U1.56 (AUD_OUT); no longer U6.7 (IO1)
- net Green_2: now also U1.51 (I2C_SDA1); no longer U6.10 (IO3)
- net Green_3: now also U1.52 (AUD_LRCLK); no longer U6.12 (IO5)
- net Green_4: now also U1.17 (UART_TX1); no longer U6.14 (IO7)
- net INT_1: now also U1.16 (I2C_INT), U4.6 (INT)
- net SCL: now also J?.5 (SCL)
- net SDA: now also J?.6 (SDA)
- net SPI_CS: now also J?.10 (~{SSEL})
- net SPI_MISO: now also J?.7 (MISO)
- net SPI_MOSI: now also J?.8 (MOSI)
- net SPI_SCK: now also J?.9 (SCK)
- net yellow_1: now also U1.54 (AUD_IN); no longer U6.6 (IO0)
- net yellow_2: now also U1.53 (I2C_SCL1); no longer U6.9 (IO2)
- net yellow_3: now also U1.50 (AUD_BCLK); no longer U6.11 (IO4)
- net yellow_4: now also U1.19 (UART_RX1); no longer U6.13 (IO6)
- net RESET: now reaches U1.6 (RESET)
- no-connect marks 51 -> 54
Other:
- moved on the sheet: J?, R2

Commit message: k
Parts:
- removed C3: 22u, Capacitor_SMD:C_0805_2012Metric, symbol Device:C_Small
- removed R1: 10k, Resistor_SMD:R_0603_1608Metric, symbol Device:R_Small
- gave numbers to parts that had none: 2
Connections:
- net GPIO[122] is gone; now on net SPI_MOSI: P9.30 (Pin_30)
- net SPI1.D0 is gone; now on net SPI_MISO: P9.29 (Pin_29)
- net SPI1.SCLK is gone; now on net SPI_SCK: P9.31 (Pin_31)
- net SPI_CS is gone; now on net SCL: J8.10 (~{SSEL}), U1.55 (SPI_CS)
- no-connect marks 54 -> 57
Other:
- moved on the sheet: P8

Commit message: y
Parts:
- removed C1, C2: 100n, Capacitor_SMD:C_0603_1608Metric, symbol Device:C_Small
- removed TP1, TP2, TP3: TestPoint, TestPoint:TestPoint_Pad_1.5x1.5mm, symbol Connector:TestPoint
- removed U3: LIS3DHTR, digikey-footprints:VFLGA-16_3x3mm, symbol dk_Motion-Sensors-Accelerometers:LIS3DHTR
- added C? (x2): 100n, Capacitor_SMD:C_0603_1608Metric, symbol Device:C_Small
- added U?: MPU-6050, Sensor_Motion:InvenSense_QFN-24_4x4mm_P0.5mm, symbol Sensor_Motion:MPU-6050
Connections:
- net Ultra_sound_Sig is gone; now on net SDA: J1.2 (Pin_2)
- net Ultra_sound_Trig is gone; now on net SCL: J1.3 (Pin_3)
- net +3V3: now also C?.1, C?.1, U?.13 (VDD), U?.8 (VDDIO)
- net GND: now also C?.2, C?.2, U?.18 (GND)
- net INT_1: now also U?.12 (INT)
- net SCL: now also U?.23 (SCL)
- net SDA: now also U?.24 (SDA)
- net at JP1.2 (C): now also U?.9 (AD0)
Other:
- moved on the sheet: JP1

Commit message: b
Parts:
- gave numbers to parts that had none: 3
Changed lines of the file:
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@@
   (symbol (lib_id "Device:C_Small") (at 662.305 109.855 0) (unit 1)
     (in_bom yes) (on_board yes)
-    (property "Reference" "C?" (id 0) (at 662.305 107.315 0)
+    (property "Reference" "C1" (id 0) (at 662.305 107.315 0)
       (effects (font (size 1.27 1.27)) (justify left))
     )
@@
   (symbol (lib_id "Sensor_Motion:MPU-6050") (at 644.525 128.905 0) (unit 1)
     (in_bom yes) (on_board yes) (fields_autoplaced)
-    (property "Reference" "U?" (id 0) (at 646.5444 145.415 0)
+    (property "Reference" "U2" (id 0) (at 646.5444 145.415 0)
       (effects (font (size 1.27 1.27)) (justify left))
     )
@@
   (symbol (lib_id "Device:C_Small") (at 671.195 109.855 0) (unit 1)
     (in_bom yes) (on_board yes)
-    (property "Reference" "C?" (id 0) (at 671.195 107.315 0)
+    (property "Reference" "C2" (id 0) (at 671.195 107.315 0)
       (effects (font (size 1.27 1.27)) (justify left))
     )
@@
   (symbol (lib_id "power:GND") (at 671.195 113.665 0) (unit 1)
     (in_bom yes) (on_board yes) (fields_autoplaced)
-    (property "Reference" "#PWR?" (id 0) (at 671.195 120.015 0)
+    (property "Reference" "#PWR0107" (id 0) (at 671.195 120.015 0)
       (effects (font (size 1.27 1.27)) hide)
     )
@@
   (symbol (lib_id "power:GND") (at 644.525 147.955 0) (unit 1)
     (in_bom yes) (on_board yes) (fields_autoplaced)
-    (property "Reference" "#PWR?" (id 0) (at 644.525 154.305 0)
+    (property "Reference" "#PWR0104" (id 0) (at 644.525 154.305 0)
       (effects (font (size 1.27 1.27)) hide)
     )
@@
   (symbol (lib_id "power:GND") (at 662.305 113.665 0) (unit 1)
     (in_bom yes) (on_board yes) (fields_autoplaced)
-    (property "Reference" "#PWR?" (id 0) (at 662.305 120.015 0)
+    (property "Reference" "#PWR0106" (id 0) (at 662.305 120.015 0)
       (effects (font (size 1.27 1.27)) hide)
     )
@@
       (reference "#PWR0103") (unit 1) (value "GND") (footprint "")
     )
+    (path "/c805c47d-893c-4d32-8581-d87646ff7aa4"
+      (reference "#PWR0104") (unit 1) (value "GND") (footprint "")
+    )
     (path "/f16d56c6-865b-438a-8efd-5a1612e4b5b9"
       (reference "#PWR0105") (unit 1) (value "+3V3") (footprint "")
     )
+    (path "/d2a398f1-32b6-4522-bfbf-5231f70db5b8"
+      (reference "#PWR0106") (unit 1) (value "GND") (footprint "")
+    )
+    (path "/c27722be-abf9-4872-85d9-db593984e6db"
+      (reference "#PWR0107") (unit 1) (value "GND") (footprint "")
+    )
     (path "/1044e081-11a0-42c0-baa5-d143d7b83424"
       (reference "#PWR0109") (unit 1) (value "GND") (footprint "")
@@
       (reference "#PWR0149") (unit 1) (value "GND") (footprint "")
     )
-    (path "/c27722be-abf9-4872-85d9-db593984e6db"
-      (reference "#PWR?") (unit 1) (value "GND") (footprint "")
-    )
-    (path "/c805c47d-893c-4d32-8581-d87646ff7aa4"
-      (reference "#PWR?") (unit 1) (value "GND") (footprint "")
-    )
-    (path "/d2a398f1-32b6-4522-bfbf-5231f70db5b8"
-      (reference "#PWR?") (unit 1) (value "GND") (footprint "")
+    (path "/4871946a-96c8-448a-b98d-6045e52daf89"
+      (reference "C1") (unit 1) (value "100n") (footprint "Capacitor_SMD:C_0603_1608Metric")
+    )
+    (path "/ad637c85-a764-4a23-9e02-be82f8a8eeee"
+      (reference "C2") (unit 1) (value "100n") (footprint "Capacitor_SMD:C_0603_1608Metric")
     )
     (path "/4a937a5e-9652-4c3b-a1c7-0db1847317a0"
@@
       (reference "C9") (unit 1) (value "100n") (footprint "Capacitor_SMD:C_0603_1608Metric_Pad1.08x0.95mm_HandSolder")
     )
-    (path "/4871946a-96c8-448a-b98d-6045e52daf89"
-      (reference "C?") (unit 1) (value "100n") (footprint "Capacitor_SMD:C_0603_1608Metric")
-    )
-    (path "/ad637c85-a764-4a23-9e02-be82f8a8eeee"
-      (reference "C?") (unit 1) (value "100n") (footprint "Capacitor_SMD:C_0603_1608Metric")
-    )
     (path "/5f684e2b-1f68-4dcb-b64e-832bf999642a"
       (reference "FID1") (unit 1) (value "Fiducial") (footprint "Z_mycustom_footprint_lib:AI-64")
@@
       (reference "U1") (unit 1) (value "SparkFun-micromod") (footprint "Z_mycustom_footprint_lib:SparkFun-micromod-footprint")
     )
+    (path "/5e6858da-1975-4260-82a9-78d4d3031db8"
+      (reference "U2") (unit 1) (value "MPU-6050") (footprint "Sensor_Motion:InvenSense_QFN-24_4x4mm_P0.5mm")
+    )
     (path "/a665ccc3-5882-45d9-b2d4-be4ed4720477"
       (reference "U4") (unit 1) (value "BNO085-breackout") (footprint "Z_mycustom_footprint_lib:BNO085-breackout")
@@
       (reference "U6") (unit 1) (value "PCA9557PW") (footprint "Package_SO:TSSOP-16_4.4x5mm_P0.65mm")
     )
-    (path "/5e6858da-1975-4260-82a9-78d4d3031db8"
-      (reference "U?") (unit 1) (value "MPU-6050") (footprint "Sensor_Motion:InvenSense_QFN-24_4x4mm_P0.5mm")
-    )
-  )
+  )

Commit message: Update Control.kicad_sch
Parts:
- U2: LCSC (none) -> C50278
Changed lines of the file:
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@@
+      (effects (font (size 1.27 1.27)) hide)
+    )
+    (property "LCSC" "C50278" (id 4) (at 644.525 128.905 0)
       (effects (font (size 1.27 1.27)) hide)
     )

Commit message: f
Parts:
- added J9: Conn_01x07, Connector_PinHeader_2.54mm:PinHeader_1x07_P2.54mm_Vertical, symbol Connector_Generic:Conn_01x07
Connections:
- net +3V3: now also J9.7 (Pin_7); no longer J6.21 (Pin_21), J6.33 (Pin_33), J7.32 (Pin_32), J7.40 (Pin_40)
- net GND: now also J6.21 (Pin_21), J6.33 (Pin_33), J7.32 (Pin_32), J7.40 (Pin_40), J9.1 (Pin_1)
- net SCL: no longer J8.10 (~{SSEL}), U1.55 (SPI_CS)
- net SPI_MISO: now also J9.3 (Pin_3)
- net SPI_MOSI: now also J9.4 (Pin_4)
- net SPI_SCK: now also J9.5 (Pin_5)
- net CS3: now reaches U6.10 (IO3)
- net CS4: now reaches U6.11 (IO4)
- net CS1: now reaches U6.7 (IO1)
- net CS1: now also J9.6 (Pin_6)
- net CS2: now reaches U6.9 (IO2)
- net GPIO[4] renamed SPI_CS
- net SPI_CS: now also J8.10 (~{SSEL}), U1.55 (SPI_CS)
- no-connect marks 57 -> 63
Other:
- note added: "RP2040/Teensy"
- moved on the sheet: C1, C2, JP1, U2

Commit message: Update Control.kicad_sch
Parts:
- added C3: 100n, Capacitor_SMD:C_0603_1608Metric_Pad1.08x0.95mm_HandSolder, symbol Device:C_Small
- added U3: CD4052B, symbol Analog_Switch:CD4052B
Connections:
- net +5V: now also C3.1, U3.16 (VDD)
- net CS1: now also U3.10 (A); no longer J9.6 (Pin_6)
- net CS2: now also U3.9 (B)
- net CS3: now also U3.6 (INH)
- net GND: now also C3.2, U3.7 (VEE), U3.8 (VSS)
- net SPI_CS: now also U3.13 (X); no longer J8.10 (~{SSEL}), P9.17 (Pin_17)
- new net SPI_CP1: J8.10 (~{SSEL}), U3.12 (X0)
- new net SPI_CP2: P9.17 (Pin_17), U3.14 (X1)
- new net SPI_CP3: J9.6 (Pin_6), U3.15 (X2)
- new net SPI_CP4: U3.11 (X3)
- no-connect marks 63 -> 64

Commit message: Update Control.kicad_sch
Parts:
- U3: footprint (none) -> Package_SO:SOIC-16_3.9x9.9mm_P1.27mm; LCSC (none) -> C6521
Changed lines of the file:
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@@
       (effects (font (size 1.27 1.27)) (justify left))
     )
-    (property "Footprint" "" (id 2) (at 397.51 370.84 0)
+    (property "Footprint" "Package_SO:SOIC-16_3.9x9.9mm_P1.27mm" (id 2) (at 397.51 370.84 0)
       (effects (font (size 1.27 1.27)) (justify left) hide)
     )
@@
       (effects (font (size 1.27 1.27)) hide)
     )
+    (property "LCSC" "C6521" (id 4) (at 393.7 351.79 0)
+      (effects (font (size 1.27 1.27)) hide)
+    )
