File: extras/kicad/V2/Control/Control.kicad_pcb (KiCad board)
At the start: 2 copper layers, 181.3 x 110 mm, 6 parts, among them J6 left, J7 right

Commit message: f
Parts:
- added FID2: Fiducial, Z_mycustom_footprint_lib:Jetson-NANO-mechanical, F.Cu at (222.4, -71.5)
- added FID4: Fiducial, Z_mycustom_footprint_lib:RPI4B-mechanical, F.Cu at (301.7, -68.1)
Changed lines of the file:
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@@
       (net 1 "GND") (pinfunction "1") (pintype "input"))
+  )
+  (footprint "Z_mycustom_footprint_lib:Jetson-NANO-mechanical" (layer "F.Cu")
+    (at 222.4 -71.5)
+    (property "Sheetfile" "Control.kicad_sch")
+    (property "Sheetname" "")
+    (property "exclude_from_bom" "")
+    (attr exclude_from_bom)
+    (fp_text reference "FID2" (at 0 -0.5 unlocked) (layer "F.SilkS")
+      (effects (font (size 1 1) (thickness 0.15)))
+    )
+    (fp_text value "Fiducial" (at 0 1 unlocked) (layer "F.Fab")
+      (effects (font (size 1 1) (thickness 0.15)))
+    )
+    (fp_text user "${REFERENCE}" (at 0 2.5 unlocked) (layer "F.Fab")
+      (effects (font (size 1 1) (thickness 0.15)))
+    )
+    (fp_arc (start 43.4525 -32.766) (mid 43.453633 -37.066001) (end 43.457834 -32.766002) (layer "Dwgs.User") (width 0.1))
+    (fp_arc (start -42.651861 25.15) (mid -42.650806 20.849999) (end -42.646527 25.149998) (layer "Dwgs.User") (width 0.1))
+    (fp_arc (start -42.751861 -32.9) (mid -42.750806 -37.200001) (end -42.746527 -32.900002) (layer "Dwgs.User") (width 0.1))
+    (fp_arc (start 43.4525 25.234) (mid 43.453633 20.933999) (end 43.457834 25.233998) (layer "Dwgs.User") (width 0.1))
+    (fp_line (start 22.0615 2.937) (end -29.9385 2.937) (layer "Edge.Cuts") (width 0.254))
+    (fp_line (start 50.0615 38.937) (end -49.9385 38.937) (layer "Edge.Cuts") (width 0.254))
+    (fp_line (start 50.0615 -39.063) (end 31.0695 -39.063) (layer "Edge.Cuts") (width 0.254))
+    (fp_line (start -29.9385 -39.063) (end -29.9465 2.937) (layer "Edge.Cuts") (width 0.254))
+    (fp_line (start 32.0615 -39.063) (end 32.0535 2.937) (layer "Edge.Cuts") (width 0.254))
+    (fp_line (start 27.0605 2.935) (end 32.0535 2.935) (layer "Edge.Cuts") (width 0.254))
+    (fp_line (start 50.0615 -39.063) (end 50.0615 38.937) (layer "Edge.Cuts") (width 0.254))
+    (fp_line (start -29.9385 -39.063) (end -49.9385 -39.063) (layer "Edge.Cuts") (width 0.254))
+    (fp_line (start -49.9385 -39.063) (end -49.9385 38.937) (layer "Edge.Cuts") (width 0.254))
+    (fp_arc (start 27.0605 2.935) (mid 24.561138 5.480405) (end 22.060477 2.936276) (layer "Edge.Cuts") (width 0.254))
+    (fp_line (start -49.9385 -39.063) (end 50.0615 -39.063) (layer "F.CrtYd") (width 0.152))
+    (fp_line (start -49.9385 38.94) (end -49.9385 -39.063) (layer "F.CrtYd") (width 0.152))
+    (fp_line (start 50.0615 38.94) (end -49.9385 38.94) (layer "F.CrtYd") (width 0.152))
+    (fp_line (start 50.0615 -39.063) (end 50.0615 38.94) (layer "F.CrtYd") (width 0.152))
+    (pad "" np_thru_hole circle (at 43.4 23.1 270) (size 2.5 2.5) (drill 2.5) (layers F&B.Cu *.Mask))
+    (pad "" np_thru_hole circle (at -42.6385 23.037 270) (size 2.5 2.5) (drill 2.5) (layers F&B.Cu *.Mask))
+    (pad "" np_thru_hole circle (at -42.7385 -35.063 270) (size 2.5 2.5) (drill 2.5) (layers F&B.Cu *.Mask))
+    (pad "" np_thru_hole circle (at 43.45 -34.85 270) (size 2.5 2.5) (drill 2.5) (layers F&B.Cu *.Mask))
   )
   (footprint "MountingHole:MountingHole_4.3mm_M4_DIN965_Pad_TopBottom" (layer "F.Cu")
@@
       (net 1 "GND") (pinfunction "1") (pintype "input"))
   )
+  (footprint "Z_mycustom_footprint_lib:RPI4B-mechanical" (layer "F.Cu")
+    (at 301.6615 -68.063)
+    (property "Sheetfile" "Control.kicad_sch")
+    (property "Sheetname" "")
+    (property "exclude_from_bom" "")
+    (attr exclude_from_bom)
+    (fp_text reference "FID4" (at 0 -0.5 unlocked) (layer "F.SilkS")
+      (effects (font (size 1 1) (thickness 0.15)))
+    )
+    (fp_text value "Fiducial" (at 0 1 unlocked) (layer "F.Fab")
+      (effects (font (size 1 1) (thickness 0.15)))
+    )
+    (fp_text user "${REFERENCE}" (at 0 2.5 unlocked) (layer "F.Fab")
+      (effects (font (size 1 1) (thickness 0.15)))
+    )
+    (fp_line (start -27.95 42.5) (end -27.95 -42.5) (layer "F.SilkS") (width 0.254))
+    (fp_line (start 28.05 42.5) (end -27.95 42.5) (layer "F.SilkS") (width 0.254))
+    (fp_line (start -27.95 -42.5) (end 28.05 -42.5) (layer "F.SilkS") (width 0.254))
+    (fp_line (start 28.05 -42.5) (end 28.05 42.5) (layer "F.SilkS") (width 0.254))
+    (fp_line (start 28.048 -42.502) (end 28.048 42.486) (layer "F.CrtYd") (width 0.152))
+    (fp_line (start 28.048 42.486) (end -27.959 42.486) (layer "F.CrtYd") (width 0.152))
+    (fp_line (start -27.959 42.486) (end -27.959 -42.502) (layer "F.CrtYd") (width 0.152))
+    (fp_line (start -27.959 -42.502) (end 28.048 -42.502) (layer "F.CrtYd") (width 0.152))
+    (pad "" np_thru_hole circle (at -24.45 -39 270) (size 2.7 2.7) (drill 2.7) (layers F&B.Cu *.Mask))
+    (pad "" np_thru_hole circle (at -24.45 19 270) (size 2.7 2.7) (drill 2.7) (layers F&B.Cu *.Mask))
+    (pad "" np_thru_hole circle (at 24.55 19 270) (size 2.7 2.7) (drill 2.7) (layers F&B.Cu *.Mask))
+    (pad "" np_thru_hole circle (at 24.55 -39 270) (size 2.7 2.7) (drill 2.7) (layers F&B.Cu *.Mask))
+  )
   (footprint "MountingHole:MountingHole_4.3mm_M4_DIN965_Pad_TopBottom" (layer "F.Cu")

Commit message: g
Parts:
- added FID1: Fiducial, Z_mycustom_footprint_lib:AI-64, F.Cu at (152.0, 92.1)
- moved FID4 259.2 mm to (107.7, 103.9), turned to 90 degrees
- moved FID2 196.3 mm to (115.0, 92.8)
Changed lines of the file:
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@@
+    )
+  )
+  (footprint "Z_mycustom_footprint_lib:AI-64" (layer "F.Cu")
+    (at 152 92.1 180)
+    (property "Sheetfile" "Control.kicad_sch")
+    (property "Sheetname" "")
+    (property "exclude_from_bom" "")
+    (attr smd exclude_from_bom)
+    (fp_text reference "FID1" (at 0 -0.5 180 unlocked) (layer "F.SilkS")
+      (effects (font (size 1 1) (thickness 0.15)))
+    )
+    (fp_text value "Fiducial" (at 0 1 180 unlocked) (layer "F.Fab")
+      (effects (font (size 1 1) (thickness 0.15)))
+    )
+    (fp_text user "${REFERENCE}" (at 0 2.5 180 unlocked) (layer "F.Fab")
+      (effects (font (size 1 1) (thickness 0.15)))
+    )
+    (fp_rect (start -52 -41) (end 52 41) (layer "F.CrtYd") (width 0.05) (fill none))
+    (model "C:/Users/robert_alfred.kecs/Documents/KiCad/my_3D_models/random_from_online/BeagleBone_AI-64_Rev_B1_3D_220826.stp"
+      (offset (xyz -227 -242 20))
+      (scale (xyz 1 1 1))
+      (rotate (xyz 0 0 0))
     )
   )
@@
   )
   (footprint "Z_mycustom_footprint_lib:Jetson-NANO-mechanical" (layer "F.Cu")
-    (at 222.4 -71.5)
+    (at 115 92.8)
     (property "Sheetfile" "Control.kicad_sch")
     (property "Sheetname" "")
@@
       (effects (font (size 1 1) (thickness 0.15)))
     )
+    (fp_line (start -29.9385 -39.063) (end -29.9465 2.937) (layer "F.SilkS") (width 0.254))
+    (fp_line (start 27.0605 2.935) (end 32.0535 2.935) (layer "F.SilkS") (width 0.254))
+    (fp_line (start 50.0615 -39.063) (end 50.0615 38.937) (layer "F.SilkS") (width 0.254))
+    (fp_line (start 32.0615 -39.063) (end 32.0535 2.937) (layer "F.SilkS") (width 0.254))
+    (fp_line (start 50.0615 38.937) (end -49.9385 38.937) (layer "F.SilkS") (width 0.254))
+    (fp_line (start 22.0615 2.937) (end -29.9385 2.937) (layer "F.SilkS") (width 0.254))
+    (fp_line (start -29.9385 -39.063) (end -49.9385 -39.063) (layer "F.SilkS") (width 0.254))
+    (fp_line (start 50.0615 -39.063) (end 32.0615 -39.063) (layer "F.SilkS") (width 0.254))
+    (fp_line (start -49.9385 -39.063) (end -49.9385 38.937) (layer "F.SilkS") (width 0.254))
+    (fp_arc (start 27.0605 2.935) (mid 24.561138 5.480405) (end 22.060477 2.936276) (layer "F.SilkS") (width 0.254))
     (fp_arc (start 43.4525 -32.766) (mid 43.453633 -37.066001) (end 43.457834 -32.766002) (layer "Dwgs.User") (width 0.1))
+    (fp_arc (start 43.4525 25.234) (mid 43.453633 20.933999) (end 43.457834 25.233998) (layer "Dwgs.User") (width 0.1))
+    (fp_arc (start -42.751861 -32.9) (mid -42.750806 -37.200001) (end -42.746527 -32.900002) (layer "Dwgs.User") (width 0.1))
     (fp_arc (start -42.651861 25.15) (mid -42.650806 20.849999) (end -42.646527 25.149998) (layer "Dwgs.User") (width 0.1))
-    (fp_arc (start -42.751861 -32.9) (mid -42.750806 -37.200001) (end -42.746527 -32.900002) (layer "Dwgs.User") (width 0.1))
-    (fp_arc (start 43.4525 25.234) (mid 43.453633 20.933999) (end 43.457834 25.233998) (layer "Dwgs.User") (width 0.1))
-    (fp_line (start 22.0615 2.937) (end -29.9385 2.937) (layer "Edge.Cuts") (width 0.254))
-    (fp_line (start 50.0615 38.937) (end -49.9385 38.937) (layer "Edge.Cuts") (width 0.254))
-    (fp_line (start 50.0615 -39.063) (end 31.0695 -39.063) (layer "Edge.Cuts") (width 0.254))
-    (fp_line (start -29.9385 -39.063) (end -29.9465 2.937) (layer "Edge.Cuts") (width 0.254))
-    (fp_line (start 32.0615 -39.063) (end 32.0535 2.937) (layer "Edge.Cuts") (width 0.254))
-    (fp_line (start 27.0605 2.935) (end 32.0535 2.935) (layer "Edge.Cuts") (width 0.254))
-    (fp_line (start 50.0615 -39.063) (end 50.0615 38.937) (layer "Edge.Cuts") (width 0.254))
-    (fp_line (start -29.9385 -39.063) (end -49.9385 -39.063) (layer "Edge.Cuts") (width 0.254))
-    (fp_line (start -49.9385 -39.063) (end -49.9385 38.937) (layer "Edge.Cuts") (width 0.254))
-    (fp_arc (start 27.0605 2.935) (mid 24.561138 5.480405) (end 22.060477 2.936276) (layer "Edge.Cuts") (width 0.254))
+    (fp_line (start 50.0615 38.94) (end -49.9385 38.94) (layer "F.CrtYd") (width 0.152))
     (fp_line (start -49.9385 -39.063) (end 50.0615 -39.063) (layer "F.CrtYd") (width 0.152))
+    (fp_line (start 50.0615 -39.063) (end 50.0615 38.94) (layer "F.CrtYd") (width 0.152))
     (fp_line (start -49.9385 38.94) (end -49.9385 -39.063) (layer "F.CrtYd") (width 0.152))
-    (fp_line (start 50.0615 38.94) (end -49.9385 38.94) (layer "F.CrtYd") (width 0.152))
-    (fp_line (start 50.0615 -39.063) (end 50.0615 38.94) (layer "F.CrtYd") (width 0.152))
     (pad "" np_thru_hole circle (at 43.4 23.1 270) (size 2.5 2.5) (drill 2.5) (layers F&B.Cu *.Mask))
+    (pad "" np_thru_hole circle (at 43.45 -34.85 270) (size 2.5 2.5) (drill 2.5) (layers F&B.Cu *.Mask))
+    (pad "" np_thru_hole circle (at -42.7385 -35.063 270) (size 2.5 2.5) (drill 2.5) (layers F&B.Cu *.Mask))
     (pad "" np_thru_hole circle (at -42.6385 23.037 270) (size 2.5 2.5) (drill 2.5) (layers F&B.Cu *.Mask))
-    (pad "" np_thru_hole circle (at -42.7385 -35.063 270) (size 2.5 2.5) (drill 2.5) (layers F&B.Cu *.Mask))
-    (pad "" np_thru_hole circle (at 43.45 -34.85 270) (size 2.5 2.5) (drill 2.5) (layers F&B.Cu *.Mask))
   )
   (footprint "MountingHole:MountingHole_4.3mm_M4_DIN965_Pad_TopBottom" (layer "F.Cu")
@@
   )
   (footprint "Z_mycustom_footprint_lib:RPI4B-mechanical" (layer "F.Cu")
-    (at 301.6615 -68.063)
+    (at 107.7 103.9 90)
     (property "Sheetfile" "Control.kicad_sch")
     (property "Sheetname" "")
     (property "exclude_from_bom" "")
     (attr exclude_from_bom)
-    (fp_text reference "FID4" (at 0 -0.5 unlocked) (layer "F.SilkS")
-      (effects (font (size 1 1) (thickness 0.15)))
-    )
-    (fp_text value "Fiducial" (at 0 1 unlocked) (layer "F.Fab")
-      (effects (font (size 1 1) (thickness 0.15)))
-    )
-    (fp_text user "${REFERENCE}" (at 0 2.5 unlocked) (layer "F.Fab")
+    (fp_text reference "FID4" (at 0 -0.5 90 unlocked) (layer "F.SilkS")
+      (effects (font (size 1 1) (thickness 0.15)))
+    )
+    (fp_text value "Fiducial" (at 0 1 90 unlocked) (layer "F.Fab")
+      (effects (font (size 1 1) (thickness 0.15)))
+    )
+    (fp_text user "${REFERENCE}" (at 0 2.5 90 unlocked) (layer "F.Fab")
       (effects (font (size 1 1) (thickness 0.15)))
     )
@@
     (fp_line (start -27.959 42.486) (end -27.959 -42.502) (layer "F.CrtYd") (width 0.152))
     (fp_line (start -27.959 -42.502) (end 28.048 -42.502) (layer "F.CrtYd") (width 0.152))
-    (pad "" np_thru_hole circle (at -24.45 -39 270) (size 2.7 2.7) (drill 2.7) (layers F&B.Cu *.Mask))
-    (pad "" np_thru_hole circle (at -24.45 19 270) (size 2.7 2.7) (drill 2.7) (layers F&B.Cu *.Mask))
-    (pad "" np_thru_hole circle (at 24.55 19 270) (size 2.7 2.7) (drill 2.7) (layers F&B.Cu *.Mask))
-    (pad "" np_thru_hole circle (at 24.55 -39 270) (size 2.7 2.7) (drill 2.7) (layers F&B.Cu *.Mask))
+    (pad "" np_thru_hole circle (at -24.45 -39) (size 2.7 2.7) (drill 2.7) (layers F&B.Cu *.Mask))
+    (pad "" np_thru_hole circle (at -24.45 19) (size 2.7 2.7) (drill 2.7) (layers F&B.Cu *.Mask))
+    (pad "" np_thru_hole circle (at 24.55 19) (size 2.7 2.7) (drill 2.7) (layers F&B.Cu *.Mask))
+    (pad "" np_thru_hole circle (at 24.55 -39) (size 2.7 2.7) (drill 2.7) (layers F&B.Cu *.Mask))
   )
   (footprint "MountingHole:MountingHole_4.3mm_M4_DIN965_Pad_TopBottom" (layer "F.Cu")

Commit message: t
Parts:
- added U1: SparkFun-micromod, Z_mycustom_footprint_lib:SparkFun-micromod-footprint, F.Cu at (256.9, 120.0)

Commit message: g
Parts:
- added C1: 100n, Capacitor_SMD:C_0603_1608Metric, F.Cu at (184.7, -25.3)
- added C2: 100n, Capacitor_SMD:C_0603_1608Metric, F.Cu at (188.9, -28.5)
- added C3: 22u, Capacitor_SMD:C_0805_2012Metric, F.Cu at (163.1, -43.4)
- added J1: Ultrasonic Ranging, Connector_PinHeader_2.54mm:PinHeader_1x04_P2.54mm_Vertical, F.Cu at (41.6, 89.6)
- added J2: Conn_01x05, Connector_PinHeader_2.54mm:PinHeader_1x05_P2.54mm_Vertical, F.Cu at (143.9, -37.9)
- added JP1: set, Jumper:SolderJumper-3_P1.3mm_Bridged12_Pad1.0x1.5mm, F.Cu at (187.4, -22.2)
- added R1: 10k, Resistor_SMD:R_0603_1608Metric, F.Cu at (167.3, -43.6)
- added TP1: TestPoint, TestPoint:TestPoint_Pad_1.5x1.5mm, F.Cu at (176.1, -33.4)
- added TP2: TestPoint, TestPoint:TestPoint_Pad_1.5x1.5mm, F.Cu at (176.1, -28.6)
- added TP3: TestPoint, TestPoint:TestPoint_Pad_1.5x1.5mm, F.Cu at (176.1, -23.6)
- added U2: ESP-01-WIFI, Connector_PinHeader_2.54mm:PinHeader_2x04_P2.54mm_Vertical, F.Cu at (148.5, -37.9)
- added U3: LIS3DHTR, digikey-footprints:VFLGA-16_3x3mm, F.Cu at (187.4, -25.7)

Commit message: F
Parts:
- added C4: 100n, Capacitor_SMD:C_0603_1608Metric_Pad1.08x0.95mm_HandSolder, F.Cu at (262.9, -30.0)
- added C5: 15p, Capacitor_SMD:C_0603_1608Metric_Pad1.08x0.95mm_HandSolder, F.Cu at (267.3, -27.5)
- added J3: Output, Connector_USB:USB_C_Receptacle_HRO_TYPE-C-31-M-12, F.Cu at (230.1, -25.8)
- added J4: Input, Connector_USB:USB_C_Receptacle_HRO_TYPE-C-31-M-12, F.Cu at (241.5, -25.8)
- added JP2: set, Jumper:SolderJumper-3_P1.3mm_Bridged12_Pad1.0x1.5mm, F.Cu at (192.8, -22.1)
- added MH1: MountingHole_3.2mm_M3_DIN965, MountingHole:MountingHole_3.2mm_M3_DIN965, B.Cu at (126.8, 126.8)
- added MH2: MountingHole_3.2mm_M3_DIN965, MountingHole:MountingHole_3.2mm_M3_DIN965, B.Cu at (126.8, 78.6)
- added MH3: MountingHole_3.2mm_M3_DIN965, MountingHole:MountingHole_3.2mm_M3_DIN965, B.Cu at (192.8, 123.7)
- added MH4: MountingHole_3.2mm_M3_DIN965, MountingHole:MountingHole_3.2mm_M3_DIN965, B.Cu at (192.8, 81.7)
- added P8: BeagleBone_Black_Header, Connector_PinHeader_2.54mm:PinHeader_2x23_P2.54mm_Vertical, B.Cu at (131.8, 125.6)
- added P9: BeagleBone_Black_Header, Connector_PinHeader_2.54mm:PinHeader_2x23_P2.54mm_Vertical, B.Cu at (131.8, 77.3)
- added R2: 2k7, Resistor_SMD:R_0603_1608Metric_Pad0.98x0.95mm_HandSolder, F.Cu at (295.6, -47.5)
- added R3: 5k1, Resistor_SMD:R_0603_1608Metric_Pad0.98x0.95mm_HandSolder, F.Cu at (276.0, -30.0)
- added R4: 5k1, Resistor_SMD:R_0603_1608Metric_Pad0.98x0.95mm_HandSolder, F.Cu at (262.9, -27.5)
- added R5: 5k1, Resistor_SMD:R_0603_1608Metric_Pad0.98x0.95mm_HandSolder, F.Cu at (304.4, -54.1)
- added R6: 5k1, Resistor_SMD:R_0603_1608Metric_Pad0.98x0.95mm_HandSolder, F.Cu at (271.6, -30.0)
- added R7: 1k, Resistor_SMD:R_0603_1608Metric_Pad0.98x0.95mm_HandSolder, F.Cu at (295.6, -45.0)
- added R8: 1k, Resistor_SMD:R_0603_1608Metric_Pad0.98x0.95mm_HandSolder, F.Cu at (267.3, -30.0)
- added R9: 1Meg, Resistor_SMD:R_0603_1608Metric_Pad0.98x0.95mm_HandSolder, F.Cu at (283.9, -33.1)
- added U4: BNO085-breackout, Z_mycustom_footprint_lib:BNO085-breackout, F.Cu at (187.0, -27.1)
- added U6: PCA9557PW, Package_SO:TSSOP-16_4.4x5mm_P0.65mm, F.Cu at (297.8, -52.0)
- moved U1 264.6 mm to (39.2, -30.3)
- moved TP1 16.8 mm to (191.8, -27.3)
- moved TP2 13.2 mm to (188.6, -32.8)
- moved TP3 12.8 mm to (184.5, -33.3)
- moved FID4 1.65 mm to (107.8, 102.2)

Commit message: r
Parts:
- added C6: 100n, Capacitor_SMD:C_0603_1608Metric_Pad1.08x0.95mm_HandSolder, F.Cu at (99.3, -28.4)
- added C7: 22u, Capacitor_SMD:C_0805_2012Metric, F.Cu at (90.9, -21.7)
- added C8: 100n, Capacitor_SMD:C_0603_1608Metric_Pad1.08x0.95mm_HandSolder, F.Cu at (95.3, -21.9)
- added C9: 100n, Capacitor_SMD:C_0603_1608Metric_Pad1.08x0.95mm_HandSolder, F.Cu at (99.6, -23.4)
- added R10: 10k, Resistor_SMD:R_0603_1608Metric, F.Cu at (99.5, -20.9)
- added R11: 10k, Resistor_SMD:R_0603_1608Metric, F.Cu at (103.5, -25.9)
- added R12: 120, Resistor_SMD:R_0603_1608Metric_Pad0.98x0.95mm_HandSolder, F.Cu at (99.3, -25.9)
- added R13: 120, Resistor_SMD:R_0603_1608Metric_Pad0.98x0.95mm_HandSolder, F.Cu at (103.6, -28.4)
- added U5: TJA1042T-3, Package_SO:SOIC-8_3.9x4.9mm_P1.27mm, F.Cu at (92.9, -26.4)
- moved U1 0.21 mm to (39.1, -30.5)
Connections:
- C4 pad 1: Net-(C4-Pad1) -> +3V3
- J1 pad 2: /Sig -> /Ultra_sound_Sig
- J1 pad 3: /Trig -> /Ultra_sound_Trig
- J6 pad 19: /Blue_2 -> +3V3
- J6 pad 21: /Black_2 -> +3V3
- J6 pad 31: /Blue_1 -> +3V3
- J6 pad 33: /Black_1 -> +3V3
- J7 pad 30: /Blue_4 -> +3V3
- J7 pad 32: /Black_4 -> +3V3
- J7 pad 38: /Blue_3 -> +3V3
- J7 pad 40: /Black_3 -> +3V3
- P8 pad 1: (no net) -> GND
- P8 pad 10: (no net) -> /GPIO[68]
- P8 pad 11: (no net) -> /GPIO[45]
- P8 pad 12: (no net) -> /GPIO[44]
- P8 pad 13: (no net) -> /GPIO[23]
- P8 pad 14: (no net) -> /GPIO[26]
- P8 pad 15: (no net) -> /GPIO[47]
- P8 pad 16: (no net) -> /GPIO[46]
- P8 pad 17: (no net) -> /GPIO[27]
- P8 pad 18: (no net) -> /GPIO[65]
- P8 pad 19: (no net) -> /GPIO[22]
- P8 pad 2: (no net) -> GND
- P8 pad 20: (no net) -> /MMC1.CMD
- P8 pad 21: (no net) -> /MMC1.CLK
- P8 pad 22: (no net) -> /MMC1.DAT[5]
- P8 pad 23: (no net) -> /MMC1.DAT[4]
- P8 pad 24: (no net) -> /MMC1.DAT[1]
- P8 pad 25: (no net) -> /MMC1.DAT[0]
- P8 pad 26: (no net) -> /LCD.PCLK
- P8 pad 27: (no net) -> /LCD.VSYNC
- P8 pad 28: (no net) -> /GPIO[61]
- P8 pad 29: (no net) -> /LCD.HSYNC
- P8 pad 3: (no net) -> /MMC1.DAT[6]
- P8 pad 30: (no net) -> /LCD.AC_BIAS_E
- P8 pad 31: (no net) -> /LCD.DATA[14]
- P8 pad 32: (no net) -> /LCD.DATA[15]
- P8 pad 33: (no net) -> /LCD.DATA[13]
- P8 pad 34: (no net) -> /LCD.DATA[11]
- P8 pad 35: (no net) -> /LCD.DATA[8]
- P8 pad 36: (no net) -> /LCD.DATA[10]
- P8 pad 37: (no net) -> /LCD.DATA[6]
- P8 pad 38: (no net) -> /LCD.DATA[9]
- P8 pad 39: (no net) -> /LCD.DATA[4]
- P8 pad 4: (no net) -> /MMC1.DAT[7]
- P8 pad 40: (no net) -> /LCD.DATA[7]
- P8 pad 41: (no net) -> /LCD.DATA[2]
- P8 pad 42: (no net) -> /LCD.DATA[5]
- P8 pad 43: (no net) -> /LCD.DATA[0]
- P8 pad 44: (no net) -> /LCD.DATA[3]
- P8 pad 45: (no net) -> GND
- P8 pad 46: (no net) -> /LCD.DATA[1]
- P8 pad 5: (no net) -> /MMC1.DAT[2]
- P8 pad 6: (no net) -> /MMC1.DAT[3]
- P8 pad 7: (no net) -> /GPIO[66]
- P8 pad 8: (no net) -> /GPIO[67]
- P8 pad 9: (no net) -> /GPIO[69]
- P9 pad 1: (no net) -> GND
- P9 pad 10: (no net) -> /~{SYS_RESET}
- P9 pad 11: (no net) -> /GPIO[30]
- P9 pad 12: (no net) -> /GPIO[60]
- P9 pad 13: (no net) -> /GPIO[31]
- P9 pad 14: (no net) -> /GPIO[40]
- P9 pad 15: (no net) -> /GPIO[48]
- P9 pad 16: (no net) -> /GPIO[51]
- P9 pad 17: (no net) -> /GPIO[4]
- P9 pad 18: (no net) -> /GPIO[5]
- P9 pad 19: (no net) -> /I2C2.SCL
- P9 pad 2: (no net) -> GND
- P9 pad 20: (no net) -> /I2C2.SDA
- P9 pad 21: (no net) -> /GPIO[3]
- P9 pad 22: (no net) -> /GPIO[2]
- P9 pad 23: (no net) -> /GPIO[49]
- P9 pad 24: (no net) -> /GPIO[15]
- P9 pad 25: (no net) -> /GPIO[117]
- P9 pad 26: (no net) -> /GPIO[14]
- P9 pad 27: (no net) -> /GPIO[125]
- P9 pad 28: (no net) -> /SPI1.CS0
- P9 pad 29: (no net) -> /SPI1.D0
- P9 pad 30: (no net) -> /GPIO[122]
- P9 pad 31: (no net) -> /SPI1.SCLK
- P9 pad 32: (no net) -> +1V8
- P9 pad 33: (no net) -> /AIN4
- P9 pad 34: (no net) -> GND
- P9 pad 35: (no net) -> /AIN6
- P9 pad 36: (no net) -> /AIN5
- P9 pad 37: (no net) -> /AIN2
- P9 pad 38: (no net) -> /AIN3
- P9 pad 39: (no net) -> /AIN0
- P9 pad 40: (no net) -> /AIN1
- P9 pad 41: (no net) -> /GPIO[20]
- P9 pad 42: (no net) -> /GPIO[7]
- P9 pad 43: (no net) -> GND
- P9 pad 44: (no net) -> GND
- P9 pad 45: (no net) -> GND
- P9 pad 46: (no net) -> GND
- P9 pad 9: (no net) -> /PWR_BUT
- R2 pad 1: Net-(C4-Pad1) -> +3V3
- U1 pad 12: unconnected-(U1-Pad12) -> SDA
- U1 pad 14: unconnected-(U1-Pad14) -> SCL
- U1 pad 16: unconnected-(U1-Pad16) -> INT
- U1 pad 3: unconnected-(U1-Pad3) -> D2+
- U1 pad 40: unconnected-(U1-Pad40) -> /INT_1
- U1 pad 41: unconnected-(U1-Pad41) -> /CAN_RX
- U1 pad 42: unconnected-(U1-Pad42) -> /INT_2
- U1 pad 43: unconnected-(U1-Pad43) -> /CAN_TX
- U1 pad 44: unconnected-(U1-Pad44) -> /Ultra_sound_Trig
- U1 pad 46: unconnected-(U1-Pad46) -> /Ultra_sound_Sig
- U1 pad 47: unconnected-(U1-Pad47) -> /CAN_STB
- U1 pad 48: unconnected-(U1-Pad48) -> AIN1_1
- U1 pad 49: unconnected-(U1-Pad49) -> BIN2_1
- U1 pad 5: unconnected-(U1-Pad5) -> D2-
- U1 pad 50: unconnected-(U1-Pad50) -> AIN2_1
- U1 pad 51: unconnected-(U1-Pad51) -> BIN1_1
- U1 pad 52: unconnected-(U1-Pad52) -> PWMA_1
- U1 pad 53: unconnected-(U1-Pad53) -> PWMA_2
- U1 pad 54: unconnected-(U1-Pad54) -> AIN2_2
- U1 pad 55: unconnected-(U1-Pad55) -> BIN2_2
- U1 pad 56: unconnected-(U1-Pad56) -> BIN1_2
- U1 pad 57: unconnected-(U1-Pad57) -> PWMB_2
- U1 pad 58: unconnected-(U1-Pad58) -> PWMB_1
- U1 pad 59: unconnected-(U1-Pad59) -> +3V3
- U1 pad 60: unconnected-(U1-Pad60) -> AIN1_2
- U1 pad 61: unconnected-(U1-Pad61) -> +3V3
- U1 pad 63: unconnected-(U1-Pad63) -> +3V3
- U1 pad 65: unconnected-(U1-Pad65) -> +3V3
- U1 pad 67: unconnected-(U1-Pad67) -> +3V3
- U1 pad 69: unconnected-(U1-Pad69) -> +3V3
- U1 pad 71: unconnected-(U1-Pad71) -> +3V3
- U1 pad 73: unconnected-(U1-Pad73) -> +3V3
- U6 pad 10: unconnected-(U6-Pad10) -> /Green_2
- U6 pad 11: unconnected-(U6-Pad11) -> /yellow_3
- U6 pad 12: unconnected-(U6-Pad12) -> /Green_3
- U6 pad 13: unconnected-(U6-Pad13) -> /yellow_4
- U6 pad 14: unconnected-(U6-Pad14) -> /Green_4
- U6 pad 16: Net-(C4-Pad1) -> +3V3
- U6 pad 6: unconnected-(U6-Pad6) -> /yellow_1
- U6 pad 7: unconnected-(U6-Pad7) -> /Green_1
- U6 pad 9: unconnected-(U6-Pad9) -> /yellow_2
