File: extras/kicad/V2/Control/Control.kicad_pcb (KiCad board)
At the start: 2 copper layers, 181.3 x 110 mm, 52 parts, among them J1 Ultrasonic Ranging, J2 Conn_01x05, J3 Output, J4 Input, J6 left, J7 right, P8 BeagleBone_Black_Header, P9 BeagleBone_Black_Header, U1 SparkFun-micromod, U2 ESP-01-WIFI, U3 LIS3DHTR, U4 BNO085-breackout, U5 TJA1042T-3, U6 PCA9557PW

Commit message: h
Parts:
- moved U1 19.8 mm to (20.0, -35.9)
Changed lines of the file:
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@@
   (net 200 "/CAN_STB")
   (footprint "Z_mycustom_footprint_lib:SparkFun-micromod-footprint" (layer "F.Cu")
-    (at 39.095 -30.5125)
+    (at 19.985 -35.8625)
     (property "Sheetfile" "Control.kicad_sch")
     (property "Sheetname" "")
@@
     (fp_arc (start 10.883614 -12.0415) (mid 12.657311 -11.285145) (end 13.388855 -9.501066) (layer "F.SilkS") (width 0.254))
     (fp_arc (start -12.011386 -9.5015) (mid -11.267437 -11.297551) (end -9.471386 -12.0415) (layer "F.SilkS") (width 0.254))
-    (fp_arc (start 13.389614 8.2945) (mid 12.651813 10.068874) (end 10.882752 10.819321) (layer "F.SilkS") (width 0.254))
+    (fp_arc (start 13.389614 8.2945) (mid 12.651812 10.06887) (end 10.882752 10.819321) (layer "F.SilkS") (width 0.254))
     (fp_arc (start -9.505386 10.8185) (mid -11.279706 10.062522) (end -12.011614 8.278139) (layer "F.SilkS") (width 0.254))
     (fp_line (start 13.388614 10.8185) (end -12.011386 10.8185) (layer "F.CrtYd") (width 0.152))
