File: extras/kicad/V2/Control/ControlSam.kicad_pcb (KiCad board)
At the start: 2 copper layers, 181.3 x 110 mm, 58 parts, among them J1 Ultrasonic Ranging, J2 Conn_01x05, J3 Output, J4 Input, J6 left, J7 right, P8 BeagleBone_Black_Header, P9 BeagleBone_Black_Header, U1 SparkFun-micromod, U2 ESP-01-WIFI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

Commit message: Added larger M.2 & Mikro click board footprints
Parts:
- moved FID2 7.62 mm to (124.5, 91.4)
- moved U4 5.08 mm to (58.4, 91.4)

Commit message: Update ControlSam.kicad_pcb
Parts:
- removed the REF** at (191.8, 77.5)
- removed the REF** at (209.8, 104.1)
- removed the REF** at (211.8, 86.0)
- added ?: , clipboard:59991624-16fe-4338-965a-cadb35774389, F.Cu at (119.4, 86.6)
- added ?: , clipboard:0e790692-d2c4-4edd-a5fc-d9b2ca1ca32a, F.Cu at (212.3, 96.6)
- added ?: , clipboard:0e790692-d2c4-4edd-a5fc-d9b2ca1ca32a, F.Cu at (212.3, 63.6)
- added REF**: USB_C_Receptacle_HRO_TYPE-C-31-M-12, Connector_USB:USB_C_Receptacle_HRO_TYPE-C-31-M-12, F.Cu at (96.5, 55.9)
- moved R2 280.1 mm to (54.2, 94.5)
- moved R5 280.1 mm to (62.9, 87.9)
- moved R7 280.1 mm to (54.2, 97.0)
- moved U6 280.1 mm to (56.4, 90.0)
- moved J3 177.6 mm to (172.7, 142.2)
- moved J4 177.6 mm to (184.1, 142.3)
- moved U1 156.8 mm to (95.4, 101.6), turned to 90 degrees
- moved C2 145.5 mm to (80.2, 68.3)
- moved JP1 145.5 mm to (78.7, 74.6)
- moved U3 145.5 mm to (78.7, 71.1)
- moved JP2 145.5 mm to (84.2, 74.7)
- moved TP1 145.5 mm to (83.2, 69.5)
- moved TP2 145.5 mm to (80.0, 64.0)
- moved TP3 145.5 mm to (75.8, 63.5)
- moved C1 145.5 mm to (76.0, 71.5)
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