File: extras/kicad/V2/Control/ControlSam.kicad_pcb (KiCad board)
At the start: 2 copper layers, 181.3 x 110 mm, 59 parts, among them J1 Ultrasonic Ranging, J2 Conn_01x05, J3 Output, J4 Input, J6 left, J7 right, P8 BeagleBone_Black_Header, P9 BeagleBone_Black_Header, U1 SparkFun-micromod, U2 ESP-01-WIFI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

Commit message: Update ControlSam.kicad_pcb
Parts:
- removed J1: Ultrasonic Ranging, Connector_PinHeader_2.54mm:PinHeader_1x04_P2.54mm_Vertical
- added REF**: TestPoint_2Pads_Pitch2.54mm_Drill0.8mm, TestPoint:TestPoint_2Pads_Pitch2.54mm_Drill0.8mm, F.Cu at (193.0, 142.2)
Changed lines of the file:
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@@
     (pad "BLT" thru_hole circle (at -4 21.5 90) (size 6 6) (drill 3.8) (layers *.Mask "F.Cu" "In1.Cu" "B.Cu")
       (solder_mask_margin 0.1))
+    (model "${KIPRJMOD}/3D/MicroMod_Processor_Board.step"
+      (offset (xyz -148 -113 4))
+      (scale (xyz 1 1 1))
+      (rotate (xyz 0 -180 180))
+    )
   )
   (footprint "Connector_PinHeader_2.54mm:PinHeader_1x05_P2.54mm_Vertical" (layer "F.Cu")
@@
     )
     (fp_rect (start -52 -41) (end 52 41) (layer "F.CrtYd") (width 0.05) (fill none))
-    (model "${DOWN}/BeagleBone_AI-64_Rev_B1_3D_220826.stp"
+    (model "${KIPRJMOD}/3D/BeagleBone_AI-64_Rev_B1_3D_220826.stp" hide
       (offset (xyz -227 -242 20))
-      (scale (xyz 1 1 1))
-      (rotate (xyz 0 0 0))
-    )
-  )
-  (footprint "Connector_PinHeader_2.54mm:PinHeader_1x04_P2.54mm_Vertical" (layer "F.Cu")
-    (at -22.86 66.04)
-    (descr "Through hole straight pin header, 1x04, 2.54mm pitch, single row")
-    (tags "Through hole pin header THT 1x04 2.54mm single row")
-    (property "Sheetfile" "Control.kicad_sch")
-    (property "Sheetname" "")
-    (attr through_hole)
-    (fp_text reference "J1" (at 0 -2.33) (layer "F.SilkS")
-      (effects (font (size 1 1) (thickness 0.15)))
-    )
-    (fp_text value " Ultrasonic Ranging" (at 0 9.95) (layer "F.Fab")
-      (effects (font (size 1 1) (thickness 0.15)))
-    )
-    (fp_text user "${REFERENCE}" (at 0 3.81 90) (layer "F.Fab")
-      (effects (font (size 1 1) (thickness 0.15)))
-    )
-    (fp_line (start -1.33 0) (end -1.33 -1.33) (layer "F.SilkS") (width 0.12))
-    (fp_line (start 1.33 1.27) (end 1.33 8.95) (layer "F.SilkS") (width 0.12))
-    (fp_line (start -1.33 8.95) (end 1.33 8.95) (layer "F.SilkS") (width 0.12))
-    (fp_line (start -1.33 1.27) (end -1.33 8.95) (layer "F.SilkS") (width 0.12))
-    (fp_line (start -1.33 1.27) (end 1.33 1.27) (layer "F.SilkS") (width 0.12))
-    (fp_line (start -1.33 -1.33) (end 0 -1.33) (layer "F.SilkS") (width 0.12))
-    (fp_line (start -1.8 -1.8) (end -1.8 9.4) (layer "F.CrtYd") (width 0.05))
-    (fp_line (start -1.8 9.4) (end 1.8 9.4) (layer "F.CrtYd") (width 0.05))
-    (fp_line (start 1.8 -1.8) (end -1.8 -1.8) (layer "F.CrtYd") (width 0.05))
-    (fp_line (start 1.8 9.4) (end 1.8 -1.8) (layer "F.CrtYd") (width 0.05))
-    (fp_line (start -1.27 8.89) (end -1.27 -0.635) (layer "F.Fab") (width 0.1))
-    (fp_line (start 1.27 -1.27) (end 1.27 8.89) (layer "F.Fab") (width 0.1))
-    (fp_line (start -0.635 -1.27) (end 1.27 -1.27) (layer "F.Fab") (width 0.1))
-    (fp_line (start 1.27 8.89) (end -1.27 8.89) (layer "F.Fab") (width 0.1))
-    (fp_line (start -1.27 -0.635) (end -0.635 -1.27) (layer "F.Fab") (width 0.1))
-    (pad "1" thru_hole rect (at 0 0) (size 1.7 1.7) (drill 1) (layers *.Cu *.Mask)
-      (net 1 "GND") (pinfunction "Pin_1") (pintype "passive"))
-    (pad "2" thru_hole oval (at 0 2.54) (size 1.7 1.7) (drill 1) (layers *.Cu *.Mask)
-      (net 12 "/Ultra_sound_Sig") (pinfunction "Pin_2") (pintype "passive"))
-    (pad "3" thru_hole oval (at 0 5.08) (size 1.7 1.7) (drill 1) (layers *.Cu *.Mask)
-      (net 13 "/Ultra_sound_Trig") (pinfunction "Pin_3") (pintype "passive"))
-    (pad "4" thru_hole oval (at 0 7.62) (size 1.7 1.7) (drill 1) (layers *.Cu *.Mask)
-      (net 4 "+3V3") (pinfunction "Pin_4") (pintype "passive"))
-    (model "${KICAD6_3DMODEL_DIR}/Connector_PinHeader_2.54mm.3dshapes/PinHeader_1x04_P2.54mm_Vertical.wrl"
-      (offset (xyz 0 0 0))
       (scale (xyz 1 1 1))
       (rotate (xyz 0 0 0))
@@
     (pad "S1" thru_hole oval (at 4.32 -3.13 180) (size 1 2.1) (drill oval 0.6 1.7) (layers *.Cu *.Mask))
     (pad "S1" thru_hole oval (at 4.32 1.05 180) (size 1 1.6) (drill oval 0.6 1.2) (layers *.Cu *.Mask))
-    (model "${KICAD6_3DMODEL_DIR}/Connector_USB.3dshapes/USB_C_Receptacle_HRO_TYPE-C-31-M-12.wrl"
-      (offset (xyz 0 0 0))
-      (scale (xyz 1 1 1))
-      (rotate (xyz 0 0 0))
+    (model "/home/sam/Downloads/2200mAh LiPo.stp"
+      (offset (xyz -37.5 31.5 -227.5))
+      (scale (xyz 1 1 1))
+      (rotate (xyz 90 0 0))
     )
   )
@@
           ) (width 0.12) (fill yes))
       ))
+    (model "/home/sam/Desktop/rosmo/smartcar_shield/extras/kicad/V2/Power/Power.step"
+      (offset (xyz -3.5 -7 -30))
+      (scale (xyz 1 1 1))
+      (rotate (xyz 180 180 90))
+    )
   )
   (footprint "Capacitor_SMD:C_0805_2012Metric" (layer "F.Cu")
@@
     (pad "15" thru_hole circle (at -1.27 -6.35 90) (size 1.778 1.778) (drill 0.914) (layers F&B.Cu *.Mask))
     (pad "16" thru_hole circle (at -1.27 -3.81 90) (size 1.778 1.778) (drill 0.914) (layers F&B.Cu *.Mask))
+    (model "/home/sam/Downloads/Mikrobus-.step"
+      (offset (xyz -13 14.5 4.5))
+      (scale (xyz 1 1 1))
+      (rotate (xyz 0 0 0))
+    )
   )
   (footprint "Z_mycustom_footprint_lib:Jetson-NANO-mechanical" (layer "F.Cu")
@@
     (pad "" np_thru_hole circle (at -42.7385 -35.063 270) (size 2.5 2.5) (drill 2.5) (layers F&B.Cu *.Mask))
     (pad "" np_thru_hole circle (at -42.6385 23.037 270) (size 2.5 2.5) (drill 2.5) (layers F&B.Cu *.Mask))
-    (model "${KIPRJMOD}/3D/Jetson nano_fixed.step" hide
+    (model "${KIPRJMOD}/3D/Jetson nano_fixed.step"
       (offset (xyz -46 -20.5 9.5))
       (scale (xyz 1 1 1))
@@
     (pad "" np_thru_hole circle (at 24.55 19 180) (size 2.7 2.7) (drill 2.7) (layers F&B.Cu *.Mask))
     (pad "" np_thru_hole circle (at 24.55 -39 180) (size 2.7 2.7) (drill 2.7) (layers F&B.Cu *.Mask))
-    (model "${KIPRJMOD}/3D/Raspberry Pi 4 Model B.STEP"
+    (model "${KIPRJMOD}/3D/Raspberry Pi 4 Model B.STEP" hide
       (offset (xyz 0 0 11))
       (scale (xyz 1 1 1))
@@
     (pad "12" thru_hole circle (at -5.661386 -9.5015 180) (size 1.524 1.524) (drill 1.016) (layers F&B.Cu *.Mask)
       (net 160 "unconnected-(U4-Pad12)") (pinfunction "BT") (pintype "input+no_connect"))
+    (model "${KIPRJMOD}/3D/BNO85.step"
+      (opacity 0.4700)      (offset (xyz -148 105.5 5.5))
+      (scale (xyz 1 1 1))
+      (rotate (xyz 0 0 0))
+    )
   )
   (footprint "Package_SO:TSSOP-16_4.4x5mm_P0.65mm" (layer "F.Cu")
@@
     (pad "15" thru_hole circle (at -1.27 -6.35 90) (size 1.778 1.778) (drill 0.914) (layers F&B.Cu *.Mask))
     (pad "16" thru_hole circle (at -1.27 -3.81 90) (size 1.778 1.778) (drill 0.914) (layers F&B.Cu *.Mask))
+    (model "/home/sam/Downloads/Mikrobus-.step"
+      (offset (xyz -13 14 4.5))
+      (scale (xyz 1 1 1))
+      (rotate (xyz 0 0 0))
+    )
   )
   (footprint "Resistor_SMD:R_0603_1608Metric_Pad0.98x0.95mm_HandSolder" (layer "F.Cu")
@@
     (pad "S1" thru_hole oval (at -4.32 -3.13) (size 1 2.1) (drill oval 0.6 1.7) (layers *.Cu *.Mask)
       (net 137 "Net-(C5-Pad1)") (pinfunction "SHIELD") (pintype "passive"))
-    (model "${KICAD6_3DMODEL_DIR}/Connector_USB.3dshapes/USB_C_Receptacle_HRO_TYPE-C-31-M-12.wrl"
-      (offset (xyz 0 0 0))
-      (scale (xyz 1 1 1))
-      (rotate (xyz 0 0 0))
+    (model "/home/sam/Desktop/dc_gear_motor_12V_500rpm.STEP"
+      (offset (xyz -2.5 -6.5 -61.5))
+      (scale (xyz 1 1 1))
+      (rotate (xyz -180 0 -90))
     )
   )
@@
     )
   )
+  (footprint "TestPoint:TestPoint_2Pads_Pitch2.54mm_Drill0.8mm" (layer "F.Cu")
+    (at 193.04 142.24)
+    (descr "Test point with 2 pins, pitch 2.54mm, drill diameter 0.8mm")
+    (tags "CONN DEV")
+    (attr exclude_from_pos_files exclude_from_bom)
+    (fp_text reference "REF**" (at 1.3 -2) (layer "F.SilkS")
+      (effects (font (size 1 1) (thickness 0.15)))
+    )
+    (fp_text value "TestPoint_2Pads_Pitch2.54mm_Drill0.8mm" (at 1.27 2) (layer "F.Fab")
+      (effects (font (size 1 1) (thickness 0.15)))
+    )
+    (fp_text user "${REFERENCE}" (at 1.3 -2) (layer "F.Fab")
+      (effects (font (size 1 1) (thickness 0.15)))
+    )
+    (fp_line (start 3.07 0.9) (end -0.53 0.9) (layer "F.SilkS") (width 0.15))
+    (fp_line (start 3.07 -0.9) (end 3.57 -0.4) (layer "F.SilkS") (width 0.15))
+    (fp_line (start -1.03 0.4) (end -1.03 -0.4) (layer "F.SilkS") (width 0.15))
+    (fp_line (start -0.53 0.9) (end -1.03 0.4) (layer "F.SilkS") (width 0.15))
+    (fp_line (start -0.53 -0.9) (end 3.07 -0.9) (layer "F.SilkS") (width 0.15))
+    (fp_line (start 3.57 0.4) (end 3.07 0.9) (layer "F.SilkS") (width 0.15))
+    (fp_line (start 3.57 -0.4) (end 3.57 0.4) (layer "F.SilkS") (width 0.15))
+    (fp_line (start -1.03 -0.4) (end -0.53 -0.9) (layer "F.SilkS") (width 0.15))
+    (fp_line (start -0.65 -1.15) (end -1.3 -0.5) (layer "F.CrtYd") (width 0.05))
+    (fp_line (start -1.3 -0.5) (end -1.3 0.5) (layer "F.CrtYd") (width 0.05))
+    (fp_line (start 3.15 1.15) (end 3.8 0.5) (layer "F.CrtYd") (width 0.05))
+    (fp_line (start -0.65 1.15) (end 3.15 1.15) (layer "F.CrtYd") (width 0.05))
+    (fp_line (start 3.8 0.5) (end 3.8 -0.5) (layer "F.CrtYd") (width 0.05))
+    (fp_line (start -1.3 0.5) (end -0.65 1.15) (layer "F.CrtYd") (width 0.05))
+    (fp_line (start 3.15 -1.15) (end -0.65 -1.15) (layer "F.CrtYd") (width 0.05))
+    (fp_line (start 3.8 -0.5) (end 3.15 -1.15) (layer "F.CrtYd") (width 0.05))
+    (pad "1" thru_hole circle (at 0 0) (size 1.4 1.4) (drill 0.8) (layers *.Cu *.Mask))
+    (pad "2" thru_hole circle (at 2.54 0) (size 1.4 1.4) (drill 0.8) (layers *.Cu *.Mask))
+    (model "/home/sam/Desktop/RodaOmni 60 mm.stp"
+      (offset (xyz -15 -16 -60.5))
+      (scale (xyz 1 1 1))
+      (rotate (xyz 90 0 -90))
+    )
+  )
   (footprint "Package_SO:SOIC-8_3.9x4.9mm_P1.27mm" (layer "F.Cu")
     (at 115.52 57.88)
@@
     (pad "S1" thru_hole oval (at -4.32 -3.13) (size 1 2.1) (drill oval 0.6 1.7) (layers *.Cu *.Mask)
       (net 149 "unconnected-(J4-PadS1)") (pinfunction "SHIELD") (pintype "passive+no_connect"))
-    (model "${KICAD6_3DMODEL_DIR}/Connector_USB.3dshapes/USB_C_Receptacle_HRO_TYPE-C-31-M-12.wrl"
-      (offset (xyz 0 0 0))
-      (scale (xyz 1 1 1))
-      (rotate (xyz 0 0 0))
-    )
-  )
+    (model "/home/sam/Desktop/37 mm DC Geared Motor Mounting Bracket.STEP"
+      (offset (xyz -9.5 -7 -57))
+      (scale (xyz 1 1 1))
+      (rotate (xyz -90 180 90))
+    )
+  )

Commit message: Idea for Mikro
Rough PCB & Schematic
Parts:
- removed J2: Conn_01x05, Connector_PinHeader_2.54mm:PinHeader_1x05_P2.54mm_Vertical
- removed the REF** at (55.9, 127.1)
- removed U2: ESP-01-WIFI, Connector_PinHeader_2.54mm:PinHeader_2x04_P2.54mm_Vertical
- added REF**: PinSocket_1x08_P2.54mm_Vertical, Connector_PinSocket_2.54mm:PinSocket_1x08_P2.54mm_Vertical, F.Cu at (69.3, 126.7)
- added REF**: PinSocket_1x08_P2.54mm_Vertical, Connector_PinSocket_2.54mm:PinSocket_1x08_P2.54mm_Vertical, F.Cu at (264.2, 119.4)
- added REF**: PinSocket_1x08_P2.54mm_Vertical, Connector_PinSocket_2.54mm:PinSocket_1x08_P2.54mm_Vertical, F.Cu at (251.5, 101.6)
- added REF**: PinSocket_1x08_P2.54mm_Vertical, Connector_PinSocket_2.54mm:PinSocket_1x08_P2.54mm_Vertical, F.Cu at (248.9, 83.8)
- added REF**: PinSocket_1x07_P2.54mm_Vertical, Connector_PinSocket_2.54mm:PinSocket_1x07_P2.54mm_Vertical, F.Cu at (93.2, 44.6)
- added REF**: PinSocket_1x08_P2.54mm_Vertical, Connector_PinSocket_2.54mm:PinSocket_1x08_P2.54mm_Vertical, F.Cu at (259.1, 43.2)
- added REF**: PinSocket_1x08_P2.54mm_Vertical, Connector_PinSocket_2.54mm:PinSocket_1x08_P2.54mm_Vertical, F.Cu at (69.5, 59.0)
- added REF**: PinHeader_2x05_P2.54mm_Horizontal, Connector_PinHeader_2.54mm:PinHeader_2x05_P2.54mm_Horizontal, F.Cu at (97.3, 145.1)
- added REF*I2C*: PinSocket_1x04_P2.54mm_Vertical, Connector_PinSocket_2.54mm:PinSocket_1x04_P2.54mm_Vertical, F.Cu at (215.9, 91.4)
- added REF*I2C*: PinSocket_1x04_P2.54mm_Vertical, Connector_PinSocket_2.54mm:PinSocket_1x04_P2.54mm_Vertical, F.Cu at (43.2, 88.9)
- moved REF** 290.3 mm to (254.1, 67.3)
- moved REF** 70.3 mm to (-15.9, 63.5)
- moved ? 43.4 mm to (181.4, 126.9), turned to -90 degrees
- moved ? 37.0 mm to (181.4, 83.8), turned to -90 degrees
- moved U1 2.50 mm to (97.9, 101.6)
Other:
- board text added: "3V3"
- board text added: "5V"
- board text added: "7Pin SPI for connecting SBC"
- board text added: "AN"
- board text added: "BACK 1"
- board text added: "BACK 2"
- board text added: "CS"
- board text added: "GND"
- board text added: "INT"
- board text added: "PWM"
- board text added: "PinSocket_1x08_P2.54mm_Vertical"
- board text added: "RST"
- board text added: "RX"
- board text added: "SCK"
- board text added: "SCL"
- board text added: "SDA"
- board text added: "SDI"
- board text added: "SDO"
- board text added: "TX"
- board text added: "UEXT for connecting WiFi/ Peripherals"
- board text removed: "5pin Breakout Garden I2C @3.3V"
- board text removed: "7Pin Breakout Garden SPI @5v"
