File: extras/kicad/V2/Control/ControlSam.kicad_sch (KiCad schematic)
At the start: 55 parts, among them J1 Ultrasonic Ranging, J2 Conn_01x05, J3 Output, J4 Input, J6 left, J7 right, J8 UEXT_Host, J9 Conn_01x07, P8 BeagleBone_Black_Header, P9 BeagleBone_Black_Header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

Commit message: Add files via upload
Parts:
- J?: value BACK 2 Conn_01x08_Female -> MIKRO_3 BACK 2 Conn_01x08_Female
- J?: value BACK 1 Conn_01x08_Female -> MIKRO_2 BACK (right) 1
- J?: value FRONT -> MIKRO_1 FRONT (left)
Connections:
- net TXD: now reaches J8.3 (TXD)
- net RXD: now reaches J8.4 (RXD)
- no-connect marks 63 -> 62

Commit message: Add files via upload
Parts:
- removed J? (x2): Conn_01x08_Female, symbol Connector:Conn_01x08_Female
- removed J?: MIKRO_3 BACK 2 Conn_01x08_Female, symbol Connector:Conn_01x08_Female
- removed J?: MIKRO_2 BACK (right) 1, symbol Connector:Conn_01x08_Female
- added J?: MIKRO_2 (top), symbol Connector:Conn_01x08_Female
- added J?: MIKRO_3 REAR (bottom), symbol Connector:Conn_01x08_Female
- added Mikro? (x2): Conn_01x08_Female, symbol Connector:Conn_01x08_Female
- J?: value MIKRO_1 FRONT (left) -> MIKRO_1 FRONT (long)
- gave numbers to parts that had none: 1
Connections:
- net CS3: now also J?.3 (Pin_3), J?.3 (Pin_3)
- net CS4: now also J?.3 (Pin_3)
- net GND: now also J?.8 (Pin_8), J?.8 (Pin_8), J?.8 (Pin_8)
- net SPI_MISO: now also J?.5 (Pin_5), J?.5 (Pin_5), J?.5 (Pin_5)
- net SPI_MOSI: now also J?.6 (Pin_6), J?.6 (Pin_6), J?.6 (Pin_6)
- net SPI_SCK: now also J?.4 (Pin_4), J?.4 (Pin_4), J?.4 (Pin_4)
- net AN_1: now reaches J?.1 (Pin_1)
- net RST_1: now reaches J?.2 (Pin_2)
- net 3v3: now reaches J?.7 (Pin_7)
- net 3v3: now also J?.7 (Pin_7), J?.7 (Pin_7)
- new net AN3: J?.1 (Pin_1)
- new net AN_2: J?.1 (Pin_1)
- new net RST_2: J?.2 (Pin_2)
- new net RST_3: J?.2 (Pin_2)
- no-connect marks 62 -> 61
Other:
- moved on the sheet: C4, H1, H2, H3, H4, R2, R7, R8, U6
